File: OS-IMS-master/PCB_IMS/1_Spacers/1a_Spacers.brd (EAGLE design)
At the start: 710 x 535 mm, 0 parts

Commit message: chore: update boards on pcbway requests
Other:
- board size 710 x 535 mm -> 667.3 x 492.1 mm
Changed lines of the file:
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@@
 <setting verticaltext="up"/>
 </settings>
-<grid distance="2" unitdist="mm" unit="mm" style="lines" multiple="1" display="yes" altdistance="0.025" altunitdist="inch" altunit="inch"/>
+<grid distance="0.01" unitdist="mm" unit="mm" style="lines" multiple="1" display="yes" altdistance="0.025" altunitdist="inch" altunit="inch"/>
 <layers>
 <layer number="1" name="Top" color="4" fill="1" visible="yes" active="yes"/>
@@
 <wire x1="-579.4486125" y1="-34.175240625" x2="-579.4486125" y2="-69.227240625" width="0.254" layer="49"/>
 <wire x1="-579.4486125" y1="-69.227240625" x2="-537.9966125" y2="-69.202240625" width="0.254" layer="49"/>
-<wire x1="83.9533875" y1="84.047759375" x2="83.9533875" y2="49.12820625" width="0.254" layer="20"/>
-<wire x1="83.9533875" y1="84.1747625" x2="42.5263875" y2="84.2747625" width="0.254" layer="20"/>
-<wire x1="42.532728125" y1="77.8215625" x2="42.554825" y2="42.78045" width="0.254" layer="20"/>
-<wire x1="83.953390625" y1="42.82275625" x2="83.953390625" y2="49.17275625" width="0.254" layer="20"/>
-<wire x1="42.579271875" y1="77.752759375" x2="42.580159375" y2="84.06655625" width="0.254" layer="20"/>
 <wire x1="-495.9966125" y1="-69.202240625" x2="-495.9966125" y2="-62.852240625" width="0.254" layer="49"/>
 <wire x1="-495.9966125" y1="-62.852240625" x2="-496.0466125" y2="-62.877240625" width="0.254" layer="49"/>
@@
 <wire x1="-621.4486125" y1="-34.175240625" x2="-621.4486125" y2="-69.227240625" width="0.254" layer="49"/>
 <wire x1="-621.4486125" y1="-69.227240625" x2="-579.9966125" y2="-69.202240625" width="0.254" layer="49"/>
-<hole x="35.8573875" y="78.078759375" drill="6.985"/>
-<hole x="6.6473875" y="78.078759375" drill="6.985"/>
-<hole x="6.6473875" y="48.868759375" drill="6.985"/>
-<hole x="35.8573875" y="48.868759375" drill="6.985"/>
-<wire x1="41.9533875" y1="84.047759375" x2="41.9533875" y2="49.12820625" width="0.254" layer="20"/>
-<wire x1="41.9533875" y1="84.1747625" x2="0.5263875" y2="84.2747625" width="0.254" layer="20"/>
-<wire x1="0.579271875" y1="84.06655625" x2="0.579271875" y2="42.78045" width="0.254" layer="20"/>
-<wire x1="41.953390625" y1="42.82275625" x2="41.953390625" y2="49.17275625" width="0.254" layer="20"/>
-<hole x="21.26739375" y="63.481878125" drill="31.75"/>
 <wire x1="-537.9966125" y1="-111.202240625" x2="-537.9966125" y2="-104.852240625" width="0.254" layer="49"/>
 <wire x1="-537.9966125" y1="-104.852240625" x2="-538.0466125" y2="-104.877240625" width="0.254" layer="49"/>
@@
 <wire x1="-579.4486125" y1="-76.175240625" x2="-579.4486125" y2="-111.227240625" width="0.254" layer="49"/>
 <wire x1="-579.4486125" y1="-111.227240625" x2="-537.9966125" y2="-111.202240625" width="0.254" layer="49"/>
-<wire x1="83.9533875" y1="42.047759375" x2="83.9533875" y2="7.12820625" width="0.254" layer="20"/>
-<wire x1="83.9533875" y1="42.1747625" x2="42.5263875" y2="42.2747625" width="0.254" layer="20"/>
-<wire x1="42.532728125" y1="35.8215625" x2="42.554825" y2="0.78045" width="0.254" layer="20"/>
-<wire x1="83.953390625" y1="0.82275625" x2="83.953390625" y2="7.17275625" width="0.254" layer="20"/>
-<wire x1="42.579271875" y1="35.752759375" x2="42.580159375" y2="42.06655625" width="0.254" layer="20"/>
 <wire x1="-495.9966125" y1="-111.202240625" x2="-495.9966125" y2="-104.852240625" width="0.254" layer="49"/>
 <wire x1="-495.9966125" y1="-104.852240625" x2="-496.0466125" y2="-104.877240625" width="0.254" layer="49"/>
@@
 <wire x1="-621.4486125" y1="-76.175240625" x2="-621.4486125" y2="-111.227240625" width="0.254" layer="49"/>
 <wire x1="-621.4486125" y1="-111.227240625" x2="-579.9966125" y2="-111.202240625" width="0.254" layer="49"/>
-<wire x1="41.9533875" y1="42.047759375" x2="41.9533875" y2="7.12820625" width="0.254" layer="20"/>
-<wire x1="41.9533875" y1="42.1747625" x2="0.5263875" y2="42.2747625" width="0.254" layer="20"/>
-<wire x1="0.579271875" y1="42.06655625" x2="0.579271875" y2="0.78045" width="0.254" layer="20"/>
-<wire x1="41.953390625" y1="0.82275625" x2="41.953390625" y2="7.17275625" width="0.254" layer="20"/>
+<wire x1="41.3" y1="41.3" x2="41.3" y2="0" width="0.254" layer="20"/>
+<wire x1="41.3" y1="41.3" x2="0" y2="41.3" width="0.254" layer="20"/>
+<wire x1="0" y1="41.3" x2="0" y2="0" width="0.254" layer="20"/>
 <wire x1="-537.9966125" y1="-153.202240625" x2="-537.9966125" y2="-146.852240625" width="0.254" layer="49"/>
 <wire x1="-537.9966125" y1="-146.852240625" x2="-538.0466125" y2="-146.877240625" width="0.254" layer="49"/>
@@
 <wire x1="-624" y1="-69.5" x2="-200.907653125" y2="-69.608846875" width="0.1524" layer="46"/>
 <wire x1="-623" y1="-405.5" x2="-199.800790625" y2="-405.60885" width="0.1524" layer="46"/>
-<hole x="35.8573875" y="36.079859375" drill="6.985"/>
-<hole x="6.6473875" y="36.079859375" drill="6.985"/>
-<hole x="6.6473875" y="6.869859375" drill="6.985"/>
-<hole x="35.8573875" y="6.869859375" drill="6.985"/>
-<hole x="21.26739375" y="21.482978125" drill="31.75"/>
-<hole x="77.8562875" y="78.078759375" drill="6.985"/>
-<hole x="48.6462875" y="78.078759375" drill="6.985"/>
-<hole x="48.6462875" y="48.868759375" drill="6.985"/>
-<hole x="77.8562875" y="48.868759375" drill="6.985"/>
-<hole x="63.26629375" y="63.481878125" drill="31.75"/>
-<hole x="77.8562875" y="36.079859375" drill="6.985"/>
-<hole x="48.6462875" y="36.079859375" drill="6.985"/>
-<hole x="48.6462875" y="6.869859375" drill="6.985"/>
-<hole x="77.8562875" y="6.869859375" drill="6.985"/>
-<hole x="63.26629375" y="21.482978125" drill="31.75"/>
-<wire x1="0.60121875" y1="42.73775" x2="41.92649375" y2="42.73775" width="0.254" layer="20"/>
-<wire x1="41.92649375" y1="42.73775" x2="41.9755125" y2="42.78676875" width="0.1524" layer="20"/>
-<wire x1="42.60011875" y1="42.73775" x2="83.92539375" y2="42.73775" width="0.254" layer="20"/>
-<wire x1="0.60121875" y1="0.73885" x2="41.92649375" y2="0.73885" width="0.254" layer="20"/>
-<wire x1="42.60011875" y1="0.73885" x2="83.92539375" y2="0.73885" width="0.254" layer="20"/>
+<hole x="35.2273875" y="35.309859375" drill="6.985"/>
+<hole x="6.0173875" y="35.309859375" drill="6.985"/>
+<hole x="6.0173875" y="6.099859375" drill="6.985"/>
+<hole x="35.2273875" y="6.099859375" drill="6.985"/>
+<hole x="20.63739375" y="20.712978125" drill="31.75"/>
+<wire x1="0" y1="0" x2="41.3" y2="0" width="0.254" layer="20"/>
 </plain>
 <attributes>
