File: OS-IMS-master/PCB_IMS/2_Electrodes/2a_Electrodes.brd (EAGLE design)
At the start: 484.8 x 419.7 mm, 0 parts

Commit message: chore: update boards on pcbway requests
Routing:
- net S$142: track 78.7 -> 0.00 mm
- net S$90: track 78.7 -> 0.00 mm
- net S$84: track 78.7 -> 0.00 mm
- net S$82: track 78.7 -> 0.00 mm
- net S$154: track 78.7 -> 0.00 mm
- net S$148: track 78.7 -> 0.00 mm
- net S$140: track 78.7 -> 0.00 mm
- net S$138: track 78.7 -> 0.00 mm
- net S$132: track 78.7 -> 0.00 mm
- net S$130: track 78.7 -> 0.00 mm
- net S$124: track 78.7 -> 0.00 mm
- net S$122: track 78.7 -> 0.00 mm
- net S$100: track 78.7 -> 0.00 mm
- net S$98: track 78.7 -> 0.00 mm
- net S$92: track 78.7 -> 0.00 mm
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Other:
- board size 484.8 x 419.7 mm -> 47.8 x 41.4 mm
- board text removed: "1""
- board text removed: "Cut out"
