File: OS-IMS-master/PCB_IMS/5_Dtector_backplate/5_detector backplate.brd (EAGLE design)
At the start: 41.5 x 41.5 mm, 0 parts

Commit message: chore: update boards on pcbway requests
Other:
- board size 41.5 x 41.5 mm -> 663.5 x 489.5 mm
Changed lines of the file:
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@@
 <?xml version="1.0" encoding="utf-8"?>
 <!DOCTYPE eagle SYSTEM "eagle.dtd">
-<eagle version="8.2.2">
+<eagle version="9.2.2">
 <drawing>
 <settings>
 <setting alwaysvectorfont="no"/>
+<setting keepoldvectorfont="yes"/>
 <setting verticaltext="up"/>
 </settings>
-<grid distance="0.000000123031" unitdist="inch" unit="inch" style="lines" multiple="1" display="yes" altdistance="0.025" altunitdist="inch" altunit="inch"/>
+<grid distance="1" unitdist="mm" unit="mm" style="lines" multiple="1" display="yes" altdistance="0.001" altunitdist="inch" altunit="inch"/>
 <layers>
 <layer number="1" name="Top" color="4" fill="1" visible="yes" active="yes"/>
@@
 <layer number="27" name="tValues" color="7" fill="1" visible="yes" active="yes"/>
 <layer number="28" name="bValues" color="7" fill="1" visible="yes" active="yes"/>
-<layer number="29" name="tStop" color="7" fill="3" visible="no" active="yes"/>
-<layer number="30" name="bStop" color="7" fill="6" visible="no" active="yes"/>
+<layer number="29" name="tStop" color="7" fill="3" visible="yes" active="yes"/>
+<layer number="30" name="bStop" color="7" fill="6" visible="yes" active="yes"/>
 <layer number="31" name="tCream" color="7" fill="4" visible="no" active="yes"/>
-<layer number="32" name="bCream" color="7" fill="5" visible="no" active="yes"/>
+<layer number="32" name="bCream" color="7" fill="5" visible="yes" active="yes"/>
 <layer number="33" name="tFinish" color="6" fill="3" visible="yes" active="yes"/>
 <layer number="34" name="bFinish" color="6" fill="6" visible="yes" active="yes"/>
@@
 <layer number="44" name="Drills" color="7" fill="1" visible="yes" active="yes"/>
 <layer number="45" name="Holes" color="7" fill="1" visible="yes" active="yes"/>
-<layer number="46" name="Milling" color="3" fill="1" visible="no" active="yes"/>
+<layer number="46" name="Milling" color="3" fill="1" visible="yes" active="yes"/>
 <layer number="47" name="Measures" color="7" fill="1" visible="yes" active="yes"/>
 <layer number="48" name="Document" color="7" fill="1" visible="yes" active="yes"/>
@@
 <board>
 <plain>
-<wire x1="-580.0466125" y1="-447.2178" x2="-580.0466125" y2="-405.6888" width="0.254" layer="49"/>
-<wire x1="-580.0466125" y1="-405.6888" x2="-621.4486125" y2="-405.6888" width="0.254" layer="49"/>
-<wire x1="-621.4486125" y1="-405.6888" x2="-621.49044375" y2="-447.217796875" width="0.254" layer="49"/>
-<wire x1="-621.49044375" y1="-447.217796875" x2="-580.0466125" y2="-447.2178" width="0.254" layer="49"/>
-<hole x="-586.1426125" y="-411.921240625" drill="6.985"/>
-<hole x="-615.3526125" y="-411.921240625" drill="6.985"/>
-<hole x="-615.3526125" y="-441.131240625" drill="6.985"/>
-<hole x="-586.1426125" y="-441.131240625" drill="6.985"/>
-<hole x="-600.73260625" y="-426.518121875" drill="7.5311"/>
-<wire x1="-580.043146875" y1="-405.6905375" x2="-621.43914375" y2="-405.69226875" width="0.254" layer="46"/>
-<wire x1="-632.74986875" y1="-405.91015625" x2="-632.77486875" y2="-405.91015625" width="0.254" layer="49"/>
-<wire x1="-621.43914375" y1="-405.69226875" x2="-621.48863125" y2="-447.224175" width="0.254" layer="46"/>
-<wire x1="-621.48863125" y1="-447.224175" x2="-580.0392" y2="-447.218946875" width="0.254" layer="46"/>
+<wire x1="41.52" y1="0" x2="41.52" y2="41.52" width="0.254" layer="20"/>
+<wire x1="41.52" y1="41.52" x2="0" y2="41.52" width="0.254" layer="20"/>
+<wire x1="0" y1="41.52" x2="0" y2="0" width="0.254" layer="20"/>
+<wire x1="0" y1="0" x2="41.52" y2="0" width="0.254" layer="20"/>
+<hole x="35.3239875" y="35.291359375" drill="6.985"/>
+<hole x="6.1139875" y="35.291359375" drill="6.985"/>
+<hole x="6.1139875" y="6.081359375" drill="6.985"/>
+<hole x="35.3239875" y="6.081359375" drill="6.985"/>
+<hole x="20.73399375" y="20.694478125" drill="7.5311"/>
+<wire x1="-580.576546875" y1="-406.4779375" x2="-621.97254375" y2="-406.47966875" width="0.254" layer="46"/>
+<wire x1="-621.97254375" y1="-406.47966875" x2="-622.02203125" y2="-448.011575" width="0.254" layer="46"/>
+<wire x1="-622.02203125" y1="-448.011575" x2="-580.5726" y2="-448.006346875" width="0.254" layer="46"/>
 <polygon width="0.254" layer="46">
-<vertex x="-580.0337375" y="-405.695521875"/>
-<vertex x="-580.0337375" y="-447.219375"/>
-<vertex x="-580.038965625" y="-447.219375"/>
+<vertex x="-580.5671375" y="-406.482921875"/>
+<vertex x="-580.5671375" y="-448.006775"/>
+<vertex x="-580.572365625" y="-448.006775"/>
 </polygon>
-<dimension x1="-615.343709375" y1="-415.413728125" x2="-615.361515625" y2="-408.428753125" x3="-626.015025" y3="-411.94841875" textsize="1.778" layer="1" dtype="diameter" unit="inch" precision="3"/>
-<dimension x1="-615.3526125" y1="-411.921240625" x2="-600.73260625" y2="-426.518121875" x3="-608.042609375" y3="-403.615796875" textsize="1.778" layer="1" dtype="horizontal" unit="inch" precision="3"/>
-<dimension x1="-621.4486125" y1="-405.6888" x2="-621.49044375" y2="-447.217796875" x3="-567.345546875" y3="-426.453296875" textsize="1.778" layer="1" dtype="vertical" unit="inch" precision="3"/>
-<dimension x1="-600.731275" y1="-422.752571875" x2="-600.7339375" y2="-430.283671875" x3="-576.168859375" y3="-426.52680625" textsize="1.778" layer="1" dtype="diameter" unit="inch" precision="3"/>
 </plain>
 <attributes>
@@
 <param name="dpMaxLengthDifference" value="10mm"/>
 <param name="dpGapFactor" value="2.5"/>
-<param name="checkGrid" value="0"/>
 <param name="checkAngle" value="0"/>
 <param name="checkFont" value="1"/>
 <param name="checkRestrict" value="1"/>
+<param name="checkStop" value="0"/>
+<param name="checkValues" value="0"/>
+<param name="checkNames" value="1"/>
+<param name="checkWireStubs" value="1"/>
+<param name="checkPolygonWidth" value="0"/>
 <param name="useDiameter" value="13"/>
 <param name="maxErrors" value="50"/>
@@
 <signals>
 </signals>
+<mfgpreviewcolors>
+<mfgpreviewcolor name="soldermaskcolor" color="0xC8008000"/>
+<mfgpreviewcolor name="silkscreencolor" color="0xFFFEFEFE"/>
+<mfgpreviewcolor name="backgroundcolor" color="0xFF282828"/>
+<mfgpreviewcolor name="coppercolor" color="0xFFFFBF00"/>
+<mfgpreviewcolor name="substratecolor" color="0xFF786E46"/>
+</mfgpreviewcolors>
 </board>
 </drawing>
