File: PCB/Divider/DividerV2.kicad_pcb (KiCad board)
At the start: 2 copper layers, 227.8 x 48 mm, 71 parts, among them J1 15kV, J2 10kV, J3 0V, J4 10kV, U1 SFH617A-1

Commit message: Pbs with footprints
Parts:
- added Electrode: Pad_for_electrode, Connector:Pad_for_electrode, F.Cu at (52.0, 58.0)
- R30: footprint Resistor_SMD:R_1206_3216Metric -> Resistor_THT:R_Axial_DIN0207_L6.3mm_D2.5mm_P15.24mm_Horizontal
- moved R47 91.9 mm to (280.0, 68.0), turned to 270 degrees
- moved R46 79.3 mm to (272.0, 68.0), turned to 270 degrees
- moved R62 77.2 mm to (284.0, 68.0), turned to 270 degrees
- moved R45 75.2 mm to (264.0, 68.0), turned to 270 degrees
- moved R60 74.5 mm to (268.0, 68.0), turned to 270 degrees
- moved R44 73.7 mm to (256.0, 68.0), turned to 270 degrees
- moved R48 70.6 mm to (288.0, 68.0), turned to 270 degrees
- moved R61 66.2 mm to (276.0, 68.0), turned to 270 degrees
- moved R59 63.7 mm to (260.0, 68.0), turned to 270 degrees
- moved R43 63.0 mm to (248.0, 68.0), turned to 270 degrees
- moved R58 59.6 mm to (252.0, 68.0), turned to 270 degrees
- moved R57 55.3 mm to (244.0, 68.0), turned to 270 degrees
- moved R36 53.6 mm to (192.0, 68.0), turned to 270 degrees
- moved R41 53.1 mm to (232.0, 68.0), turned to 270 degrees
- moved R55 52.8 mm to (228.0, 68.0), turned to 270 degrees
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Routing:
- net (no net): vias 1 -> 0

Commit message: PCB + new electrodes
Parts:
- added E1: Electr., Connector:Pad_for_electrode, F.Cu at (55.6, 44.3)
- added E10: Electr., Connector:Pad_for_electrode, F.Cu at (120.6, 46.5)
- added E11: Electr., Connector:Pad_for_electrode, F.Cu at (127.2, 44.6)
- added E12: Electr., Connector:Pad_for_electrode, F.Cu at (134.6, 43.8)
- added E13: Electr., Connector:Pad_for_electrode, F.Cu at (142.2, 43.4)
- added E14: Electr., Connector:Pad_for_electrode, F.Cu at (148.8, 41.4)
- added E15: Electr., Connector:Pad_for_electrode, F.Cu at (162.6, 50.6)
- added E16: Electr., Connector:Pad_for_electrode, F.Cu at (59.0, 107.8)
- added E17: Electr., Connector:Pad_for_electrode, F.Cu at (66.6, 106.6)
- added E18: Electr., Connector:Pad_for_electrode, F.Cu at (73.6, 105.8)
- added E19: Electr., Connector:Pad_for_electrode, F.Cu at (81.0, 107.2)
- added E2: Electr., Connector:Pad_for_electrode, F.Cu at (62.0, 44.4)
- added E20: Electr., Connector:Pad_for_electrode, F.Cu at (88.0, 106.8)
- added E21: Electr., Connector:Pad_for_electrode, F.Cu at (95.6, 107.6)
- added E22: Electr., Connector:Pad_for_electrode, F.Cu at (101.8, 107.0)
- added E23: Electr., Connector:Pad_for_electrode, F.Cu at (109.6, 106.8)
- added E24: Electr., Connector:Pad_for_electrode, F.Cu at (117.4, 107.4)
- added E25: Electr., Connector:Pad_for_electrode, F.Cu at (124.4, 107.1)
- added E26: Electr., Connector:Pad_for_electrode, F.Cu at (131.8, 106.0)
- added E27: Electr., Connector:Pad_for_electrode, F.Cu at (138.4, 107.2)
- added E28: Electr., Connector:Pad_for_electrode, F.Cu at (145.2, 107.0)
- added E29: Electr., Connector:Pad_for_electrode, F.Cu at (164.6, 80.2)
- added E3: Electr., Connector:Pad_for_electrode, F.Cu at (69.6, 44.7)
- added E4: Electr., Connector:Pad_for_electrode, F.Cu at (77.0, 45.7)
- added E5: Electr., Connector:Pad_for_electrode, F.Cu at (84.0, 44.6)
- added E6: Electr., Connector:Pad_for_electrode, F.Cu at (91.6, 45.1)
- added E7: Electr., Connector:Pad_for_electrode, F.Cu at (98.4, 45.1)
- added E8: Electr., Connector:Pad_for_electrode, F.Cu at (105.8, 45.8)
- added E9: Electr., Connector:Pad_for_electrode, F.Cu at (113.6, 46.7)
- added Electrode: Pad_for_electrode, Connector:Pad_for_electrode, F.Cu at (62.8, 58.5)
- added Electrode: Pad_for_electrode, Connector:Pad_for_electrode, F.Cu at (102.4, 93.7)
- added Electrode: Pad_for_electrode, Connector:Pad_for_electrode, F.Cu at (98.8, 58.5)
- added Electrode: Pad_for_electrode, Connector:Pad_for_electrode, F.Cu at (109.6, 93.6)
- added Electrode: Pad_for_electrode, Connector:Pad_for_electrode, F.Cu at (95.2, 93.6)
- added Electrode: Pad_for_electrode, Connector:Pad_for_electrode, F.Cu at (116.8, 93.6)
- added Electrode: Pad_for_electrode, Connector:Pad_for_electrode, F.Cu at (124.0, 93.7)
- added Electrode: Pad_for_electrode, Connector:Pad_for_electrode, F.Cu at (134.8, 58.6)
- added Electrode: Pad_for_electrode, Connector:Pad_for_electrode, F.Cu at (127.6, 58.5)
- added Electrode: Pad_for_electrode, Connector:Pad_for_electrode, F.Cu at (84.4, 58.5)
- added Electrode: Pad_for_electrode, Connector:Pad_for_electrode, F.Cu at (91.6, 58.6)
- added Electrode: Pad_for_electrode, Connector:Pad_for_electrode, F.Cu at (149.2, 58.5)
- added Electrode: Pad_for_electrode, Connector:Pad_for_electrode, F.Cu at (80.8, 93.7)
- added Electrode: Pad_for_electrode, Connector:Pad_for_electrode, F.Cu at (73.6, 93.6)
- added Electrode: Pad_for_electrode, Connector:Pad_for_electrode, F.Cu at (88.0, 93.6)
- added Electrode: Pad_for_electrode, Connector:Pad_for_electrode, F.Cu at (77.2, 58.5)
- added Electrode: Pad_for_electrode, Connector:Pad_for_electrode, F.Cu at (70.0, 58.6)
- added Electrode: Pad_for_electrode, Connector:Pad_for_electrode, F.Cu at (66.4, 93.6)
- added Electrode: Pad_for_electrode, Connector:Pad_for_electrode, F.Cu at (59.2, 93.7)
- added Electrode: Pad_for_electrode, Connector:Pad_for_electrode, F.Cu at (55.6, 58.6)
- added Electrode: Pad_for_electrode, Connector:Pad_for_electrode, F.Cu at (145.6, 93.7)
- added Electrode: Pad_for_electrode, Connector:Pad_for_electrode, F.Cu at (142.0, 58.5)
- added Electrode: Pad_for_electrode, Connector:Pad_for_electrode, F.Cu at (138.4, 93.6)
- added Electrode: Pad_for_electrode, Connector:Pad_for_electrode, F.Cu at (113.2, 58.6)
- added Electrode: Pad_for_electrode, Connector:Pad_for_electrode, F.Cu at (106.0, 58.5)
- added Electrode: Pad_for_electrode, Connector:Pad_for_electrode, F.Cu at (120.4, 58.5)
- added Electrode: Pad_for_electrode, Connector:Pad_for_electrode, F.Cu at (131.2, 93.6)
- R1, R10, R11, R12, R13, R14, R15, R16, R17, R18, R19, R2, R20, R21, R22, R23, R24, R25, R26, R27, R28, R29, R3, R4, R5, R6, R7, R8, R9: footprint LED_SMD:LED_1206_3216Metric -> Resistor_SMD:R_1206_3216Metric_Pad1.42x1.75mm_HandSolder
- moved Electrode 35.6 mm to (52.0, 93.6)
- moved J3 28.5 mm to (39.0, 91.4)
- moved J1 26.4 mm to (34.4, 101.8)
- moved J4 22.0 mm to (43.4, 104.0)
- moved R14 15.9 mm to (145.6, 80.0)
- moved R13 15.4 mm to (138.4, 80.0)
- moved R12 14.9 mm to (131.2, 80.0)
- moved C3 14.7 mm to (75.7, 24.8)
- moved R11 14.4 mm to (124.0, 80.0)
- moved R10 14.0 mm to (116.8, 80.0)
- moved R9 13.6 mm to (109.6, 80.0)
- moved R8 13.2 mm to (102.4, 80.0)
- moved R7 12.9 mm to (95.2, 80.0)
- moved R6 12.6 mm to (88.0, 80.0)
- moved R5 12.4 mm to (80.8, 80.0)
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- renumbered J4 to J2, J2 to J3, J3 to J4
Routing:
- net Net-(E1-Pad1): track 0.00 -> 10.0 mm
- net /Drift_tube: track 0.00 -> 4.01 mm

Commit message: 1st pcb done
Parts:
- removed Electrode (x28): Pad_for_electrode, Connector:Pad_for_electrode
- moved R29 126.5 mm to (178.5, 77.0), turned to 90 degrees
- moved J3 68.8 mm to (77.6, 44.3)
- moved E14 52.3 mm to (145.8, 93.6)
- moved E13 50.3 mm to (138.6, 93.6)
- moved E12 49.9 mm to (131.4, 93.6)
- moved E1 49.4 mm to (52.2, 93.6)
- moved E16 49.3 mm to (55.8, 58.6)
- moved E2 49.3 mm to (59.4, 93.6)
- moved E21 49.1 mm to (91.8, 58.6)
- moved E11 49.1 mm to (124.2, 93.6)
- moved E5 49.1 mm to (81.0, 93.6)
- moved E3 49.0 mm to (66.6, 93.6)
- moved E24 49.0 mm to (113.4, 58.6)
- moved E19 48.7 mm to (77.4, 58.6)
- moved E27 48.7 mm to (135.0, 58.6)
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- renumbered J3 to J2, J4 to J3, J2 to J4, R2 to R1, R11 to R10, R12 to R11, R13 to R12, R14 to R13, R15 to R14, R16 to R15, R17 to R16, R18 to R17, R19 to R18, R20 to R19, R3 to R2, R21 to R20, R22 to R21, R23 to R22, R24 to R23, R25 to R24, R26 to R25, R27 to R26, R28 to R27, R29 to R28, R1 to R29, R4 to R3, R5 to R4, R6 to R5, R7 to R6, R8 to R7, R9 to R8, R10 to R9
Connections:
- E1 pad 1: Net-(E1-Pad1) -> /Drift_tube
- E15 pad 1: TRI-STATE -> Net-(E15-Pad1)
- R14 pad 1: TRI-STATE -> Net-(E15-Pad1)
- R15 pad 1: Net-(E1-Pad1) -> /Drift_tube
- R29 pad 1: Net-(E1-Pad1) -> Net-(E15-Pad1)
- R29 pad 2: /Drift_tube -> TRI-STATE
Routing:
- net Net-(E17-Pad1): track 0.00 -> 22.1 mm
- net Net-(E14-Pad1): track 0.00 -> 22.0 mm
- net Net-(E7-Pad1): track 0.00 -> 22.0 mm
- net Net-(E6-Pad1): track 0.00 -> 22.0 mm
- net Net-(E24-Pad1): track 0.00 -> 22.0 mm
- net Net-(E23-Pad1): track 0.00 -> 22.0 mm
- net Net-(E19-Pad1): track 0.00 -> 22.0 mm
- net Net-(E18-Pad1): track 0.00 -> 22.0 mm
- net Net-(E12-Pad1): track 0.00 -> 22.0 mm
- net Net-(E11-Pad1): track 0.00 -> 22.0 mm
- net Net-(E2-Pad1): track 0.00 -> 22.0 mm
- net Net-(E9-Pad1): track 0.00 -> 22.0 mm
- net Net-(E8-Pad1): track 0.00 -> 22.0 mm
- net Net-(E5-Pad1): track 0.00 -> 22.0 mm
- net Net-(E4-Pad1): track 0.00 -> 22.0 mm
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