File: PCB/Divider/DividerV2.sch (KiCad schematic (older format))
At the start: 71 parts, among them U1 SFH617A-1

Commit message: Pbs with footprints
Parts:
- gave numbers to parts that had none: 4
Changed lines of the file:
@@
 	2600 6150 2750 6150
 $Comp
-L Connector:Conn_01x01_Female J?
+L Connector:Conn_01x01_Female J2
 U 1 1 5F9A8D86
 P 8850 3050
-AR Path="/5F9A8D86" Ref="J?"  Part="1"
+AR Path="/5F9A8D86" Ref="J2"  Part="1"
 AR Path="/5F465EFE/5F9A8D86" Ref="J?"  Part="1"
-F 0 "J?" H 8878 3076 50  0000 L CNN
+F 0 "J2" H 8878 3076 50  0000 L CNN
 F 1 "10kV" H 8878 2985 50  0000 L CNN
 F 2 "Connector_Pin:Pin_D1.4mm_L8.5mm_W2.8mm_FlatFork" H 8850 3050 50  0001 C CNN
@@
 $EndComp
 $Comp
-L Connector:Conn_01x01_Female J?
+L Connector:Conn_01x01_Female J3
 U 1 1 5F9A8D8C
 P 8850 3400
-AR Path="/5F9A8D8C" Ref="J?"  Part="1"
+AR Path="/5F9A8D8C" Ref="J3"  Part="1"
 AR Path="/5F465EFE/5F9A8D8C" Ref="J?"  Part="1"
-F 0 "J?" H 8878 3426 50  0000 L CNN
+F 0 "J3" H 8878 3426 50  0000 L CNN
 F 1 "0V" H 8878 3335 50  0000 L CNN
 F 2 "Connector_Pin:Pin_D1.4mm_L8.5mm_W2.8mm_FlatFork" H 8850 3400 50  0001 C CNN
@@
 $EndComp
 $Comp
-L power:GND #PWR?
+L power:GND #PWR0101
 U 1 1 5F9A8D92
 P 8450 3400
-AR Path="/5F9A8D92" Ref="#PWR?"  Part="1"
+AR Path="/5F9A8D92" Ref="#PWR0101"  Part="1"
 AR Path="/5F465EFE/5F9A8D92" Ref="#PWR?"  Part="1"
-F 0 "#PWR?" H 8450 3150 50  0001 C CNN
+F 0 "#PWR0101" H 8450 3150 50  0001 C CNN
 F 1 "GND" H 8455 3227 50  0000 C CNN
 F 2 "" H 8450 3400 50  0001 C CNN
@@
 $EndComp
 $Comp
-L Connector:Conn_01x01_Female J?
+L Connector:Conn_01x01_Female J1
 U 1 1 5F9A8D98
 P 7700 3050
-AR Path="/5F9A8D98" Ref="J?"  Part="1"
+AR Path="/5F9A8D98" Ref="J1"  Part="1"
 AR Path="/5F465EFE/5F9A8D98" Ref="J?"  Part="1"
-F 0 "J?" H 7728 3076 50  0000 L CNN
+F 0 "J1" H 7728 3076 50  0000 L CNN
 F 1 "15kV" H 7728 2985 50  0000 L CNN
 F 2 "Connector_Pin:Pin_D1.4mm_L8.5mm_W2.8mm_FlatFork" H 7700 3050 50  0001 C CNN
@@
 $EndComp
 $Comp
-L Connector:Conn_01x01_Female J?
+L Connector:Conn_01x01_Female J4
 U 1 1 5F9A8D9E
 P 7700 3500
-AR Path="/5F9A8D9E" Ref="J?"  Part="1"
+AR Path="/5F9A8D9E" Ref="J4"  Part="1"
 AR Path="/5F465EFE/5F9A8D9E" Ref="J?"  Part="1"
-F 0 "J?" H 7728 3526 50  0000 L CNN
+F 0 "J4" H 7728 3526 50  0000 L CNN
 F 1 "10kV" H 7728 3435 50  0000 L CNN
 F 2 "Connector_Pin:Pin_D1.4mm_L8.5mm_W2.8mm_FlatFork" H 7700 3500 50  0001 C CNN

Commit message: PCB + new electrodes
Parts:
- added E1, E10, E11, E12, E13, E14, E15, E16, E17, E18, E19, E2, E20, E21, E22, E23, E24, E25, E26, E27, E28, E29, E3, E4, E5, E6, E7, E8, E9: Electr., Connector:Pad_for_electrode, symbol Connector:Conn_01x01_Female
- R1, R10, R11, R12, R13, R14, R15, R16, R17, R18, R19, R2, R20, R21, R22, R23, R24, R25, R26, R27, R28, R29, R3, R4, R5, R6, R7, R8, R9: footprint LED_SMD:LED_1206_3216Metric -> Resistor_SMD:R_1206_3216Metric_Pad1.42x1.75mm_HandSolder
- R30: footprint Resistor_SMD:R_1206_3216Metric -> Resistor_THT:R_Axial_DIN0207_L6.3mm_D2.5mm_P15.24mm_Horizontal
- renumbered J4 to J2, J2 to J3, J3 to J4
Connections:
- net TRI-STATE: now also E15.1 (Pin_1)
- net at R1.1, R16.1: now also E1.1 (Pin_1)
- net at R17.1, R2.1: now also E2.1 (Pin_1)
- net at R17.2, R3.2: now also E17.1 (Pin_1)
- net at R16.2, R2.2: now also E16.1 (Pin_1)
- net at R18.1, R3.1: now also E3.1 (Pin_1)
- net at R18.2, R4.2: now also E18.1 (Pin_1)
- net at R19.1, R4.1: now also E4.1 (Pin_1)
- net at R20.1, R5.1: now also E5.1 (Pin_1)
- net at R19.2, R5.2: now also E19.1 (Pin_1)
- net at R20.2, R6.2: now also E20.1 (Pin_1)
- net at R21.1, R6.1: now also E6.1 (Pin_1)
- net at R21.2, R7.2: now also E21.1 (Pin_1)
- net at R22.1, R7.1: now also E7.1 (Pin_1)
- net at R23.1, R8.1: now also E8.1 (Pin_1)
- net at R22.2, R8.2: now also E22.1 (Pin_1)
- net at R23.2, R9.2: now also E23.1 (Pin_1)
- net at R24.1, R9.1: now also E9.1 (Pin_1)
- net at R10.2, R24.2: now also E24.1 (Pin_1)
- net at R10.1, R25.1: now also E10.1 (Pin_1)
- net at R11.1, R26.1: now also E11.1 (Pin_1)
- net at R11.2, R25.2: now also E25.1 (Pin_1)
- net at R12.2, R26.2: now also E26.1 (Pin_1)
- net at R12.1, R27.1: now also E12.1 (Pin_1)
- net at R13.2, R27.2: now also E27.1 (Pin_1)
- net at R13.1, R28.1: now also E13.1 (Pin_1)
- net at R14.1, R29.1: now also E14.1 (Pin_1)
- net at R14.2, R28.2: now also E28.1 (Pin_1)
- net at R15.2, R29.2: now also E29.1 (Pin_1)

Commit message: 1st pcb done
Parts:
- renumbered J3 to J2, J4 to J3, J2 to J4, R2 to R1, R11 to R10, R12 to R11, R13 to R12, R14 to R13, R15 to R14, R16 to R15, R17 to R16, R18 to R17, R19 to R18, R20 to R19, R3 to R2, R21 to R20, R22 to R21, R23 to R22, R24 to R23, R25 to R24, R26 to R25, R27 to R26, R28 to R27, R29 to R28, R1 to R29, R4 to R3, R5 to R4, R6 to R5, R7 to R6, R8 to R7, R9 to R8, R10 to R9
Connections:
- net Drift_tube: now also E1.1 (Pin_1), R15.1; no longer R29.2
- net TRI-STATE: now also R29.2; no longer E15.1 (Pin_1), R14.1
- new net: E15.1 (Pin_1), R14.1, R29.1
Other:
- moved on the sheet: R29
