File: PCB/Divider/DividerV2/DividerV2.kicad_pcb (KiCad board)
At the start: 2 copper layers, 227.8 x 48 mm, 100 parts, among them J1 15kV, J2 10kV, J3 0V, J4 10kV, U1 SFH617A-1

Commit message: Reorganisation
Parts:
- moved E29 24.4 mm to (149.4, 58.6)
- moved R14 15.1 mm to (149.4, 72.0), turned to 90 degrees
Routing:
- net Net-(E29-Pad1): track 0.00 -> 22.0 mm
Changed lines of the file:
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@@
   (general
     (thickness 1.6)
-    (drawings 19)
-    (tracks 106)
+    (drawings 18)
+    (tracks 110)
     (zones 0)
     (modules 100)
@@
   )
   (module Connector:Pad_for_electrode (layer F.Cu)
-    (at 163 78.9)
+    (at 149.4 58.6)
     (fp_text reference E29 (at 0.5 6.9) (layer F.SilkS) hide
       (effects (font (size 1 1) (thickness 0.15)))
@@
   )
   (module Resistor_SMD:R_1206_3216Metric_Pad1.42x1.75mm_HandSolder (layer F.Cu)
-    (at 164 68 270)
+    (at 149.4 72 90)
     (descr "Resistor SMD 1206 (3216 Metric), square (rectangular) end terminal, IPC_7351 nominal with elongated pad for handsoldering. (Body size source: http://www.tortai-tech.com/upload/download/2011102023233369053.pdf), generated with kicad-footprint-generator")
     (tags "resistor handsolder")
@@
     (fp_line (start -1.6 -0.8) (end 1.6 -0.8) (layer F.Fab) (width 0.1))
     (fp_line (start -1.6 0.8) (end -1.6 -0.8) (layer F.Fab) (width 0.1))
-    (pad 2 smd roundrect (at 1.4875 0 270) (size 1.425 1.75) (layers F.Cu F.Paste F.Mask) (roundrect_rratio 0.175439)
+    (pad 2 smd roundrect (at 1.4875 0 90) (size 1.425 1.75) (layers F.Cu F.Paste F.Mask) (roundrect_rratio 0.175439)
       (net 67 "Net-(E29-Pad1)"))
-    (pad 1 smd roundrect (at -1.4875 0 270) (size 1.425 1.75) (layers F.Cu F.Paste F.Mask) (roundrect_rratio 0.175439)
+    (pad 1 smd roundrect (at -1.4875 0 90) (size 1.425 1.75) (layers F.Cu F.Paste F.Mask) (roundrect_rratio 0.175439)
       (net 68 "Net-(E15-Pad1)"))
     (model ${KISYS3DMOD}/Resistor_SMD.3dshapes/R_1206_3216Metric.wrl
@@
   )
   (dimension 13.5 (width 0.15) (layer Dwgs.User)
-    (gr_text "13,500 mm" (at 49.7 65.25 270) (layer Dwgs.User)
+    (gr_text "13,500 mm" (at 49.7 65.25 90) (layer Dwgs.User)
       (effects (font (size 1 1) (thickness 0.15)))
     )
-    (feature1 (pts (xy 51 72) (xy 50.413579 72)))
-    (feature2 (pts (xy 51 58.5) (xy 50.413579 58.5)))
-    (crossbar (pts (xy 51 58.5) (xy 51 72)))
-    (arrow1a (pts (xy 51 72) (xy 50.413579 70.873496)))
-    (arrow1b (pts (xy 51 72) (xy 51.586421 70.873496)))
-    (arrow2a (pts (xy 51 58.5) (xy 50.413579 59.626504)))
-    (arrow2b (pts (xy 51 58.5) (xy 51.586421 59.626504)))
-  )
-  (dimension 13.5 (width 0.12) (layer Dwgs.User)
-    (gr_text "13,500 mm" (at 56.27 86.75 90) (layer Dwgs.User)
-      (effects (font (size 1 1) (thickness 0.15)))
-    )
-    (feature1 (pts (xy 52 80) (xy 55.586421 80)))
-    (feature2 (pts (xy 52 93.5) (xy 55.586421 93.5)))
-    (crossbar (pts (xy 55 93.5) (xy 55 80)))
-    (arrow1a (pts (xy 55 80) (xy 55.586421 81.126504)))
-    (arrow1b (pts (xy 55 80) (xy 54.413579 81.126504)))
-    (arrow2a (pts (xy 55 93.5) (xy 55.586421 92.373496)))
-    (arrow2b (pts (xy 55 93.5) (xy 54.413579 92.373496)))
+    (feature1 (pts (xy 48.4 58.5) (xy 48.986421 58.5)))
+    (feature2 (pts (xy 48.4 72) (xy 48.986421 72)))
+    (crossbar (pts (xy 48.4 72) (xy 48.4 58.5)))
+    (arrow1a (pts (xy 48.4 58.5) (xy 48.986421 59.626504)))
+    (arrow1b (pts (xy 48.4 58.5) (xy 47.813579 59.626504)))
+    (arrow2a (pts (xy 48.4 72) (xy 48.986421 70.873496)))
+    (arrow2b (pts (xy 48.4 72) (xy 47.813579 70.873496)))
   )
   (dimension 24 (width 0.12) (layer Dwgs.User)
@@
   (segment (start 138.6 78.5125) (end 138.6 73.2375) (width 2) (layer F.Cu) (net 66))
   (segment (start 142.2 70.5125) (end 142.2 58.5) (width 2) (layer F.Cu) (net 66))
+  (segment (start 148.525 70.5125) (end 149.4 70.5125) (width 2) (layer F.Cu) (net 67))
+  (segment (start 145.8 73.2375) (end 148.525 70.5125) (width 2) (layer F.Cu) (net 67))
+  (segment (start 145.8 78.5125) (end 145.8 73.2375) (width 2) (layer F.Cu) (net 67))
+  (segment (start 149.4 70.5125) (end 149.4 58.5) (width 2) (layer F.Cu) (net 67))
 )
