File: PCB/Divider/Complete_divider/_autosave-Divider1.kicad_pcb (KiCad board)
At the start: 2 copper layers, 103.8 x 48 mm, 56 parts, among them J1 10kV

Commit message: Divider1: Without tracks
Parts:
- added J28: Electr., Connector_Pin:Pin_D1.0mm_L10.0mm, F.Cu at (148.6, 72.0)
Connections:
- net DRIFTTUBE renamed DESOLVATION
Routing:
- net TRI-STATE: track 0.00 -> 13.5 mm
- net Net-(E3-Pad1): track 22.0 -> 12.0 mm
- net Net-(E2-Pad1): track 22.0 -> 12.0 mm
- net Net-(E27-Pad1): track 22.0 -> 12.0 mm
- net Net-(E5-Pad1): track 22.0 -> 12.0 mm
- net Net-(E4-Pad1): track 22.1 -> 17.2 mm
- net Net-(E25-Pad1): track 22.0 -> 17.3 mm
- net Net-(E9-Pad1): track 22.0 -> 17.3 mm
- net Net-(E6-Pad1): track 22.0 -> 17.3 mm
- net Net-(E21-Pad1): track 22.0 -> 17.3 mm
- net Net-(E19-Pad1): track 22.0 -> 17.3 mm
- net Net-(E16-Pad1): track 22.0 -> 17.3 mm
- net Net-(E14-Pad1): track 22.0 -> 17.3 mm
- net Net-(E8-Pad1): track 22.0 -> 17.3 mm
- net Net-(E7-Pad1): track 22.0 -> 17.3 mm
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