File: PCB/Divider/Complete_divider/Divider1.sch (KiCad schematic (older format))
At the start: 58 parts, among them J1 10kV

Commit message: Divider1: Without tracks
Parts:
- removed R14, R15: 10M, Resistor_SMD:R_1206_3216Metric_Pad1.42x1.75mm_HandSolder, symbol Device:R
- added J28: Electr., Connector_Pin:Pin_D1.0mm_L10.0mm, symbol Connector:Conn_01x01_Female
- renumbered E20 to E10, E6 to E11, E21 to E12, E7 to E13, E22 to E14, E8 to E15, E23 to E16, E9 to E17, E24 to E18, E10 to E19, E16 to E2, E25 to E20, E11 to E21, E26 to E22, E12 to E23, E27 to E24, E13 to E25, E28 to E26, E14 to E27, E29 to E28, E2 to E3, E17 to E4, E3 to E5, E18 to E6, E4 to E7, E19 to E8, E5 to E9, R16 to R1, R5 to R10, R21 to R11, R6 to R12, R22 to R13, R7 to R14, R23 to R15, R8 to R16, R24 to R17, R9 to R18, R25 to R19, R1 to R2, R10 to R20, R26 to R21, R11 to R22, R27 to R23, R12 to R24, R28 to R25, R13 to R26, R29 to R27, R17 to R3, R2 to R4, R18 to R5, R3 to R6, R19 to R7, R4 to R8, R20 to R9
Connections:
- net TRI-STATE: now also E28.1 (Pin_1), R27.2, J28.1 (Pin_1)
- net DRIFTTUBE renamed DESOLVATION

Commit message: Most parts completed
Parts:
- J1: value 10kV -> 15kV
Other:
- note added: "Source #2 \n0-15kV\n"
- note removed: "Source #2 \n0-10kV\n"
- moved on the sheet: J1
Changed lines of the file:
@@
 $EndComp
 Wire Wire Line
-	2650 3950 3100 3950
+	2650 3950 2850 3950
 $Comp
 L Connector:Conn_01x01_Female E1
@@
 Wire Wire Line
 	3100 3950 3250 3950
-Text Label 2900 3950 1    50   ~ 0
-Drift_tube
 $Comp
 L Connector:Conn_01x01_Female J1
 U 1 1 5E64177D
-P 7200 2600
+P 3300 3000
 AR Path="/5E64177D" Ref="J1"  Part="1"
 AR Path="/5F465EFE/5E64177D" Ref="J?"  Part="1"
 AR Path="/5E63F098/5E64177D" Ref="J?"  Part="1"
 AR Path="/5E6FA86A/5E64177D" Ref="J1"  Part="1"
-F 0 "J1" H 7228 2626 50  0000 L CNN
-F 1 "10kV" H 7228 2535 50  0000 L CNN
-F 2 "Connector_Pin:Pin_D1.4mm_L8.5mm_W2.8mm_FlatFork" H 7200 2600 50  0001 C CNN
-F 3 "~" H 7200 2600 50  0001 C CNN
-	1    7200 2600
+F 0 "J1" H 3328 3026 50  0000 L CNN
+F 1 "15kV" H 3328 2935 50  0000 L CNN
+F 2 "Connector_Pin:Pin_D1.4mm_L8.5mm_W2.8mm_FlatFork" H 3300 3000 50  0001 C CNN
+F 3 "~" H 3300 3000 50  0001 C CNN
+	1    3300 3000
 	1    0    0    -1
 $EndComp
-Text Notes 6900 2100 0    50   ~ 0
-Source #2 \n0-10kV\n
-Text Label 7000 2600 2    50   ~ 0
-Drift_tube
+Text Notes 3000 2500 0    50   ~ 0
+Source #2 \n0-15kV\n
 Wire Notes Line
-	7450 3050 7450 2200
+	3550 3450 3550 2600
 Wire Notes Line
-	7450 2200 6600 2200
+	3550 2600 2700 2600
 Wire Notes Line
-	6600 2200 6600 3050
+	2700 2600 2700 3450
 Wire Notes Line
-	6600 3050 7450 3050
+	2700 3450 3550 3450
 $Comp
 L Device:R R17
@@
 Wire Wire Line
 	7700 4650 7950 4650
+Wire Wire Line
+	2850 3950 2850 3000
+Wire Wire Line
+	2850 3000 3100 3000
+Connection ~ 2850 3950
+Wire Wire Line
+	2850 3950 3100 3950
 $EndSCHEMATC

Commit message: Begin PCB design
Parts:
- renumbered E1 to E29, E3 to E30, E5 to E31, E7 to E32, E9 to E33, E11 to E34, E13 to E35, E15 to E36, E17 to E37, E19 to E38, E21 to E39, E23 to E40, E25 to E41, E27 to E42, E2 to E43, E4 to E44, E6 to E45, E8 to E46, E10 to E47, E12 to E48, E14 to E49, E16 to E50, E18 to E51, E20 to E52, E22 to E53, E24 to E54, E26 to E55, E28 to E56, J1 to J2, J28 to J3, R2 to R28, R4 to R29, R6 to R30, R8 to R31, R10 to R32, R12 to R33, R14 to R34, R16 to R35, R18 to R36, R20 to R37, R22 to R38, R24 to R39, R26 to R40, R1 to R41, R3 to R42, R5 to R43, R7 to R44, R9 to R45, R11 to R46, R13 to R47, R15 to R48, R17 to R49, R19 to R50, R21 to R51, R23 to R52, R25 to R53, R27 to R54
