File: PCB/Divider/Complete_divider/Alim_and_ctr.sch (KiCad schematic (older format))
At the start: 38 parts

Commit message: New isolated alimentation design
Parts:
- removed R?: 1M, symbol Device:R
- added R?: 1K, symbol Device:R
- added U?: OPAMP, symbol pspice:OPAMP
- C?: value 470uF -> 2,2uF
- R?: value 10R 1W -> 20K
- U?: symbol symbols:Lolin32 -> Complete_divider-rescue:Lolin32-symbols
Connections:
- net labels removed: ALIMHV-
- wire segments 146 -> 147
Other:
- moved on the sheet: C?, Q?, R?, U?

Commit message: Modifications of the amplification part
Parts:
- J?: value Alim2 -> AlimHV2
Other:
- moved on the sheet: C?, Q?, R?, U?

Commit message: small changes
Parts:
- removed C?: 2,2uF, Capacitor_THT:C_Rect_L13.0mm_W8.0mm_P10.00mm_FKS3_FKP3_MKS4, symbol Device:C
- removed J?: Low voltage in, symbol Connector:Conn_01x02_Male
- removed PS?: RHV3-0512S/R20, Converter_DCDC:Converter_DCDC_XP_POWER-ITXxxxxSA_THT, symbol Converter_DCDC:ITX0503SA-H
- removed Q?: BC337, digikey-footprints:TO-39-3, symbol dk_Transistors-Bipolar-BJT-RF:2N5109
- removed R?: 20K, symbol Device:R
- removed R?: 1K, symbol Device:R
- removed U?: PC123, Package_DIP:DIP-4_W7.62mm, symbol Isolator:SFH617A-1
- removed U?: OPAMP, symbol pspice:OPAMP
- HV2: symbol HV_source:15A -> Alim_and_ctr-rescue:15A-HV_source
Connections:
- net labels removed: +12V, GNDA
- wire segments 147 -> 112
Other:
- note removed: "ISOLATED ALIM\n"
- note removed: "PWM \n"

Commit message: Voltage measure circuits
Parts:
- removed HV2: 15A, symbol Alim_and_ctr-rescue:15A-HV_source
- removed J?: AlimHV2, symbol Connector:Conn_01x02_Male
- removed R?: 100M, symbol Device:R
- removed U?: SFH617A-1, Package_DIP:DIP-4_W7.62mm, symbol Isolator:SFH617A-1
- added C?: 2,2uF, Capacitor_THT:C_Rect_L13.0mm_W8.0mm_P10.00mm_FKS3_FKP3_MKS4, symbol Device:C
- added C?: 15pF, symbol Device:C_Small
- added C?: 47uF/100V, symbol Device:CP1_Small
- added C?: 0.1nF, symbol Device:CP1_Small
- added HV?: 15A, symbol HV_source:15A
- added J?: Low voltage in, symbol Connector:Conn_01x02_Male
- added PS1: RHV2-1212S/R20, Converter_DCDC:Converter_DCDC_XP_POWER-ITXxxxxSA_THT, symbol Converter_DCDC:ITX0503SA-H
- added PS?: R12P212S/R8, Converter_DCDC:Converter_DCDC_XP_POWER-ITXxxxxSA_THT, symbol Converter_DCDC:ITX0503SA
- added Q?: BC337, digikey-footprints:TO-39-3, symbol dk_Transistors-Bipolar-BJT-RF:2N5109
- added Q?: ZVN2110A, symbol Device:Q_NMOS_DGS
- added R?: 1K, symbol Device:R
- added R?: 20K, symbol Device:R
- added R?: 5K, symbol Device:R_Small
- added R?: 50R, symbol Device:R_Small
- added U?: PC123, Package_DIP:DIP-4_W7.62mm, symbol Isolator:SFH617A-1
- added U?: LM358P, symbol pspice:OPAMP
- added U?: mEZD41501A-X, Converter_DCDC:Converter_DCDC_muRata_OKI-78SR_Horizontal, symbol Converter_DCDC:OKI-78SR-3.3_1.5-W36H-C
- added U?: 6N136S, Package_DIP:SMDIP-8_W9.53mm, symbol Isolator:6N136S
- gave numbers to parts that had none: 1
Connections:
- net labels added: +12V, +12VA, +15V, +3V3, ALIMHV1+, ALIMHV1-, DRIFT_TUBE, EOUTPIN, GATE_IN+, GATE_IN-, GATE_OUT, GNDA
- net labels removed: ALIMHV+, DRIFTTUBE
- wire segments 112 -> 187
- no-connect marks 0 -> 1
Other:
- note added: "Decoupling \nopto IC\n\n"
- note added: "GATE PULSER"
- note added: "ISOLATED ALIM\n"
- note added: "PWM \n"
- note added: "Pinouts"
- note removed: "Pinouts for Electrodes\n"
- moved on the sheet: C?, E?, J?, POT?, R?, U?

Commit message: Begin PCB design
Parts:
- removed HV?: 15A, symbol HV_source:15A
- removed J? (x2): Pinout, Connector_Pin:Pin_D1.0mm_L10.0mm, symbol Connector:Conn_01x01_Female
- removed PS?: R12P212S/R8, Converter_DCDC:Converter_DCDC_XP_POWER-ITXxxxxSA_THT, symbol Converter_DCDC:ITX0503SA
- removed Q?: FDV303N, digikey-footprints:SOT-23-3, symbol dk_Transistors-FETs-MOSFETs-Single:FDV303N
- removed U?: PC123, Package_DIP:DIP-4_W7.62mm, symbol Isolator:SFH617A-1
- removed U?: LM358P, symbol pspice:OPAMP
- removed U?: mEZD41501A-X, Converter_DCDC:Converter_DCDC_muRata_OKI-78SR_Horizontal, symbol Converter_DCDC:OKI-78SR-3.3_1.5-W36H-C
- added C10: 100uF, Capacitor_THT:CP_Radial_D5.0mm_P2.50mm, symbol Device:CP1_Small
- added C8: 100nF, Capacitor_SMD:C_0805_2012Metric, symbol Device:C_Small
- added D1: PWR LED, LED_THT:LED_D4.0mm, symbol Device:LED
- added HV2: 15A, HV_source:15A, symbol HV_source:15A
- added PS1: RHV2-1212S/R20, Isolated_converters:R8, symbol Complete_divider-rescue:ITX0503SA-H-Converter_DCDC
- added R66: R_LED, Resistor_SMD:R_0805_2012Metric, symbol Device:R_Small
- added SW1: EN switch, Connector_PinHeader_2.54mm:PinHeader_2x01_P2.54mm_Vertical, symbol Switch:SW_SPST
- added SW2: HV1 Switch, Connector_PinHeader_2.54mm:PinHeader_2x01_P2.54mm_Vertical, symbol Switch:SW_SPST
- added SW3: PWR switch, Connector_PinHeader_2.54mm:PinHeader_2x01_P2.54mm_Vertical, symbol Switch:SW_SPST
- added U2: mEZD41501A-X, Connector_JST:JST_EH_B6B-EH-A_1x06_P2.50mm_Vertical, symbol Converter_DCDC:mEZD41501A-X
- added U3: LM358, Package_DIP:DIP-8_W10.16mm_LongPads, symbol Amplifier_Operational:LM358
- added U4: CNY17-1, Package_DIP:DIP-6_W7.62mm, symbol Isolator:CNY17-1
- C4: renamed from C?; footprint Capacitor_THT:C_Rect_L13.0mm_W8.0mm_P10.00mm_FKS3_FKP3_MKS4 -> Capacitor_THT:C_Rect_L19.0mm_W8.0mm_P15.00mm_MKS4
- C5: renamed from C?; footprint (none) -> Capacitor_THT:CP_Radial_D18.0mm_P7.50mm
- C6: renamed from C?; value 0.1nF -> 100nF; footprint (none) -> Capacitor_SMD:C_0805_2012Metric
- C7: renamed from C?; footprint (none) -> Capacitor_SMD:C_0805_2012Metric
- C9: renamed from C?; footprint Capacitor_THT:C_Rect_L13.0mm_W8.0mm_P10.00mm_FKS3_FKP3_MKS4 -> Capacitor_THT:CP_Radial_D5.0mm_P2.50mm
- E57, E58, E59: renamed from E?; footprint Connector_Pin:Pin_D1.0mm_L10.0mm -> Connector_Wire:SolderWirePad_1x01_Drill2.5mm
- HV1: footprint (none) -> HV_source:G40
- J1: renamed from J?; footprint (none) -> Connector_PinHeader_2.54mm:PinHeader_2x01_P2.54mm_Vertical
- J10: renamed from J?; value Pinout -> Gate; footprint Connector_Pin:Pin_D1.0mm_L10.0mm -> Connector_Wire:SolderWirePad_1x01_Drill2.5mm
- J4, J5, J6, J7, J8: renamed from J?; footprint Connector_Pin:Pin_D1.0mm_L10.0mm -> Connector_Wire:SolderWirePad_1x01_Drill2.5mm
- POT1: renamed from POT?; footprint Potentiometer_THT:Potentiometer_ACP_CA14-H4_Horizontal -> Potentiometer_THT:Potentiometer_Bourns_3386C_Horizontal
- POT2: renamed from POT?; footprint (none) -> Potentiometer_THT:Potentiometer_Bourns_3386C_Horizontal
- PS2: renamed from PS1; footprint Converter_DCDC:Converter_DCDC_XP_POWER-ITXxxxxSA_THT -> Isolated_converters:R20; symbol Converter_DCDC:ITX0503SA-H -> Complete_divider-rescue:ITX0503SA-H-Converter_DCDC
- Q1: renamed from Q?; footprint (none) -> Transistors:S8050
- Q2: renamed from Q?; value BC337 -> S8050; footprint digikey-footprints:TO-39-3 -> Transistors:S8050
- R1, R2: renamed from R?; footprint (none) -> Resistor_SMD:R_0805_2012Metric_Pad1.15x1.40mm_HandSolder
- R3, R56, R57: renamed from R?; footprint (none) -> Resistor_SMD:R_1206_3216Metric
- R4, R64, R65: renamed from R?; footprint (none) -> Resistor_SMD:R_0805_2012Metric
- R55: renamed from R?; footprint Resistor_THT:R_Axial_DIN0207_L6.3mm_D2.5mm_P15.24mm_Horizontal -> Resistor_THT:R_Axial_DIN0204_L3.6mm_D1.6mm_P7.62mm_Horizontal
- R58: renamed from R?; value 100M -> 1M; footprint (none) -> Resistor_SMD:R_1206_3216Metric
- U1: renamed from U?; footprint Package_DIP:SMDIP-8_W9.53mm -> Package_DIP:DIP-8_W10.16mm_LongPads
- U5: renamed from U?; footprint (none) -> Dev_boards:Lolin32
- gave numbers to parts that had none: 4
Connections:
- net labels added: Gate
- net labels removed: Grid2, HV2_EN
- wire segments 187 -> 223
- no-connect marks 1 -> 26
Other:
- note added: "Contact with the\nlast electrode\n"
- note added: "GND : MCU, HV2\nGNDA : Gate\nGNDB : HV1\n"
- moved on the sheet: C3, J1, J10, R3, R55, R58, R64, R65, U5

Commit message: Components in place
Parts:
- R7: renamed from R2; footprint Resistor_SMD:R_0805_2012Metric_Pad1.15x1.40mm_HandSolder -> Resistor_SMD:R_1206_3216Metric
- renumbered E57 to E1, E58 to E2, E59 to E3, J4 to J1, J5 to J2, J6 to J3, J7 to J4, J8 to J5, J1 to J6, J10 to J7, R56 to R1, R64 to R10, R65 to R11, R66 to R12, R57 to R2, R59 to R3, R55 to R4, R58 to R5, R1 to R6, R3 to R8, R4 to R9

Commit message: HV design finished
Parts:
- removed U4: CNY17-1, Package_DIP:DIP-6_W7.62mm, symbol Isolator:CNY17-1
- added D2: Protection, Diode_THT:D_T-1_P5.08mm_Horizontal, symbol Device:D
- added F1: Fuse, Fuse:Fuse_1206_3216Metric, symbol Device:Fuse_Small
- added JP1: Jumper, Connector_PinHeader_1.00mm:PinHeader_1x02_P1.00mm_Horizontal, symbol Device:Jumper_NO_Small
- added OPTO2: CNY65AYST, OptoDevice:CNY65AYST, symbol Isolator:SFH617A-1
- added U4: MC78M15ACTG, Package_TO_SOT_THT:TO-262-3_Vertical, symbol Regulator_Linear:MC78M05_TO252
- C5: footprint Capacitor_THT:CP_Radial_D18.0mm_P7.50mm -> Capacitor_THT:CP_Radial_D12.5mm_P5.00mm
- E1: renamed from E2; value Electrode out -> Mid electrode1; footprint Connector_Wire:SolderWirePad_1x01_Drill2.5mm -> Connector_Wire:SolderWirePad_1x01_Drill1.5mm
- E2: renamed from E3; value Electrode out -> Mid electrode2; footprint Connector_Wire:SolderWirePad_1x01_Drill2.5mm -> Connector_Wire:SolderWirePad_1x01_Drill1.5mm
- J1, J2, J3, J4, J7: footprint Connector_Wire:SolderWirePad_1x01_Drill2.5mm -> Connector_Wire:SolderWirePad_1x01_Drill1.5mm
- J5: value HV out -> Last Electrode; footprint Connector_Wire:SolderWirePad_1x01_Drill2.5mm -> Connector_Wire:SolderWirePad_1x01_Drill1.5mm
- J6: value Low voltage in -> 12V in
- J8: renamed from E1; value Electrode out -> Ap Grid; footprint Connector_Wire:SolderWirePad_1x01_Drill2.5mm -> Connector_Wire:SolderWirePad_1x01_Drill1.5mm
- POT1: footprint Potentiometer_THT:Potentiometer_Bourns_3386C_Horizontal -> Potentiometer_THT:Potentiometer_Omeg_PC16BU_Vertical
- POT2: footprint Potentiometer_THT:Potentiometer_Bourns_3386C_Horizontal -> Potentiometer_THT:Potentiometer_Piher_T-16H_Single_Horizontal
- PS1, PS2: symbol Complete_divider-rescue:ITX0503SA-H-Converter_DCDC -> Complete_divider-rescue:ITX0503SA-H-Converter_DCDC-Complete_divider-rescue
- Q2: value S8050 -> ZTX1053A
- R4: renamed from R5; footprint Resistor_SMD:R_1206_3216Metric -> Resistor_SMD:R_0805_2012Metric
- renumbered U1 to OPTO1, R4 to R1, R1 to R2, R2 to R3, R3 to R5, R9 to R8, R8 to R9, U2 to U1, U3 to U2, U5 to U3
Connections:
- net +12V: now also JP1.1
- net +15V: now also OPTO2.4; no longer R9.2
- net +5V: now also U4.3 (VO)
- net GND: now also D2.2 (A), OPTO2.2, U4.2 (GND); no longer C1.2, C2.2, C3.2, C4.2, HV2.8 (HV_GND), J5.1 (Pin_1), R1.2
- net GNDA: no longer C8.2, C9.2, PS2.3 (-Vout), U1.3 (GND), U1.4 (GND), U2.4 (V-), U2.5 (+)
- net PWM: now also OPTO2.1
- net at J6.1 (Pin_1): now also F1.1; no longer SW3.2 (B)
- net at R8.1: now also R9.2, OPTO2.3; no longer R9.1
- new net: D2.1 (K), F1.2, SW3.2 (B)
- new net: JP1.2, U4.1 (VI)
- new net GNDB: C8.2, C9.2, PS2.3 (-Vout), R9.1, U1.3 (GND), U1.4 (GND), U2.4 (V-), U2.5 (+)
- new net LAST_ELECTRODE: C1.2, C2.2, C3.2, C4.2, HV2.8 (HV_GND), J5.1 (Pin_1), R1.2
- no-connect marks 26 -> 25
Other:
- moved on the sheet: C10, D1, E1, E2, J6, J8, R12, R8, R9

Commit message: Improve PCBs
Parts:
- removed OPTO1: 6N136S, Package_DIP:DIP-8_W10.16mm_LongPads, symbol Isolator:6N136S
- added C12: 0.33uF Tant., Capacitor_Tantalum_SMD:CP_EIA-3528-21_Kemet-B_Pad1.50x2.35mm_HandSolder, symbol Device:CP1
- added TP10, TP11, TP12, TP2, TP4, TP5, TP6, TP7, TP8, TP9: TestPoint, TestPoint:TestPoint_Keystone_5000-5004_Miniature, symbol Connector:TestPoint
- added U6: 6N137A, Package_DIP:DIP-8_W7.62mm_Socket, symbol 6N137A:6N137A
- Q1, Q2: footprint Transistors:S8050 -> Package_TO_SOT_THT:TO-220-3_Vertical
- U2: footprint Package_DIP:DIP-8_W10.16mm_LongPads -> Package_DIP:DIP-8_W7.62mm_Socket
Connections:
- net +12V: now also C12.1
- net +12VA: now also U6.8 (Vin)
- net +15V: now also TP7.1
- net ALIMHV1+: now also TP12.1
- net GATE_IN+: now also TP4.1
- net GATE_IN-: now also TP8.1
- net GND: now also C12.2, U6.3
- net GNDA: now also TP2.1, U6.5 (GND)
- net GNDB: now also TP11.1
- net GRID_CTRL: now also U6.2
- net at Q2.2 (B), U2.1: now also TP10.1
- net at C9.1, R8.2, U2.3 (+): now also TP9.1
- net at PS2.4 (+Vout), U1.1 (IN), U1.2 (IN): now also TP5.1
- net at C7.1, Q1.2 (G), R6.2: now also TP6.1, U6.6 (Vout)
Other:
- note added: "HV1\n"
- note added: "QUESTIONS\n- Reverse voltage protection\n- Alim de HV1 chute de tension\n- Quels cables utiliser\n- Alim 5V MCU : conflit entre les deux tension?\n\n"
- note removed: "PWM \n"
- moved on the sheet: C1, C2, C3, C8, R1, U2B, U2C, U4
