File: PCB/Divider/Complete_divider/Alim_and_ctr.kicad_pcb (KiCad board)
At the start: 2 copper layers, 193 x 130 mm, 75 parts, among them J1 Electrode in, J10 LCD2 PWR, J11 LCD1 V/I measures, J12 LCD1 PWR, J2 Electrode out, J3 HV out, J4 HV out, J5 Last Electrode, J6 12V in, J7 Gate, J8 Ap Grid, J9 LCD2 Vin, Q1 ZVN2110A, Q2 ZTX1053A, SW1 EN switch, SW2 HV1 Switch, SW3 PWR switch, U1 mEZD41501A-X, U2 LM358, U3 Lolin32, U4 MC78M15ACTG, U5 LM358P, U6 6N137A

Commit message: update
Parts:
- moved Q1 5.44 mm to (104.0, 69.0)
- moved TP6 2.00 mm to (96.0, 72.0)
Routing:
- net Net-(C7-Pad1): track 23.3 -> 20.4 mm
Changed lines of the file:
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@@
     (thickness 1.6)
     (drawings 16)
-    (tracks 171)
+    (tracks 172)
     (zones 0)
     (modules 75)
@@
   )
   (module Package_TO_SOT_THT:TO-220-3_Vertical (layer F.Cu)
-    (at 99.46 72)
+    (at 104 69)
     (descr "TO-220-3, Vertical, RM 2.54mm, see https://www.vishay.com/docs/66542/to-220-1.pdf")
     (tags "TO-220-3 Vertical RM 2.54mm")
@@
   )
   (module TestPoint:TestPoint_Keystone_5000-5004_Miniature (layer F.Cu)
-    (at 94 72)
+    (at 96 72)
     (descr "Keystone Miniature THM Test Point 5000-5004, http://www.keyelco.com/product-pdf.cfm?p=1309")
     (tags "Through Hole Mount Test Points")
@@
   (segment (start 85 63) (end 97 63) (width 1) (layer F.Cu) (net 8))
   (segment (start 77 55) (end 85 63) (width 1) (layer F.Cu) (net 8))
-  (segment (start 97 63) (end 97 67) (width 1) (layer F.Cu) (net 8))
-  (segment (start 99.46 69.46) (end 99.46 72) (width 1) (layer F.Cu) (net 8))
-  (segment (start 97 67) (end 99.46 69.46) (width 1) (layer F.Cu) (net 8))
+  (segment (start 102.73 67.57) (end 102.73 69.69) (width 1) (layer F.Cu) (net 8))
+  (segment (start 102.73 66.53) (end 102.73 67.57) (width 1) (layer F.Cu) (net 8))
+  (segment (start 99.2 63) (end 102.73 66.53) (width 1) (layer F.Cu) (net 8))
+  (segment (start 97 63) (end 99.2 63) (width 1) (layer F.Cu) (net 8))
   (via (at 70 68) (size 0.8) (drill 0.4) (layers F.Cu B.Cu) (net 9))
   (via (at 106 75) (size 0.8) (drill 0.4) (layers F.Cu B.Cu) (net 9))
@@
   (segment (start 116.88 62.5) (end 113.475 62.5) (width 1) (layer F.Cu) (net 10))
   (segment (start 112.3 59.975) (end 113 59.975) (width 1) (layer F.Cu) (net 11))
-  (segment (start 112.025 59.975) (end 112.3 59.975) (width 1) (layer F.Cu) (net 11))
-  (segment (start 102 70) (end 112.025 59.975) (width 1) (layer F.Cu) (net 11))
-  (segment (start 102 72) (end 102 70) (width 1) (layer F.Cu) (net 11))
-  (segment (start 113 59.975) (end 113 57.9375) (width 1) (layer F.Cu) (net 11))
+  (segment (start 111.595 59.975) (end 112.3 59.975) (width 1) (layer F.Cu) (net 11))
+  (segment (start 104 67.57) (end 111.595 59.975) (width 1) (layer F.Cu) (net 11))
+  (segment (start 104 69.69) (end 104 67.57) (width 1) (layer F.Cu) (net 11))
   (segment (start 116.3625 57.9375) (end 116.88 57.42) (width 1) (layer F.Cu) (net 11))
   (segment (start 113 57.9375) (end 116.3625 57.9375) (width 1) (layer F.Cu) (net 11))
+  (segment (start 113 57.9375) (end 113 59.975) (width 1) (layer F.Cu) (net 11))
   (via (at 127 143) (size 0.8) (drill 0.4) (layers F.Cu B.Cu) (net 12))
   (segment (start 127 143) (end 129 141) (width 0.7) (layer B.Cu) (net 12))
