File: PCB/Divider/Complete_divider/Alim_and_ctr.kicad_pcb (KiCad board)
At the start: 2 copper layers, 100 x 100 mm, 14 parts, among them U11 SFH617A-1

Commit message: Begin PCB design
Parts:
- removed C11, C12, C13: 4700pF 10kV, Capacitor_THT:C_Rect_L13.0mm_W8.0mm_P10.00mm_FKS3_FKP3_MKS4
- removed E29, E30: Electrode, Connector_Pin:Pin_D1.0mm_L10.0mm
- removed R101, R103: 1.5M, Resistor_SMD:R_1206_3216Metric
- removed R102: 100M, Resistor_SMD:R_1206_3216Metric
- removed R104: 500K, Resistor_THT:R_Axial_DIN0207_L6.3mm_D2.5mm_P15.24mm_Horizontal
- removed R28, R29, R30: 10M, Resistor_SMD:R_1206_3216Metric
- removed RV11: 100M, Potentiometer_THT:Potentiometer_ACP_CA14-H4_Horizontal
- removed U11: SFH617A-1, Package_DIP:DIP-4_W7.62mm
- added C1: 4700pF 10kV, Capacitor_THT:C_Rect_L13.0mm_W8.0mm_P10.00mm_FKS3_FKP3_MKS4, F.Cu at (26.6, 133.0)
- added C10: 100uF, Capacitor_THT:CP_Radial_D5.0mm_P2.50mm, F.Cu at (187.0, 59.0)
- added C2: 4700pF 10kV, Capacitor_THT:C_Rect_L13.0mm_W8.0mm_P10.00mm_FKS3_FKP3_MKS4, F.Cu at (26.9, 121.1)
- added C3: 0.22uF, Capacitor_THT:C_Rect_L13.0mm_W8.0mm_P10.00mm_FKS3_FKP3_MKS4, F.Cu at (116.0, 143.0)
- added C4: 2500pF 15 kV, Capacitor_THT:C_Rect_L19.0mm_W8.0mm_P15.00mm_MKS4, F.Cu at (33.0, 72.0)
- added C5: 47uF/100V, Capacitor_THT:CP_Radial_D18.0mm_P7.50mm, F.Cu at (143.5, 20.5)
- added C6: 100nF, Capacitor_SMD:C_0805_2012Metric, F.Cu at (132.0, 20.0)
- added C7: 15pF, Capacitor_SMD:C_0805_2012Metric, F.Cu at (128.5, 9.50)
- added C8: 100nF, Capacitor_SMD:C_0805_2012Metric, F.Cu at (130.0, 106.9)
- added C9: 2,2uF, Capacitor_THT:CP_Radial_D5.0mm_P2.50mm, F.Cu at (109.0, 122.0)
- added D1: PWR LED, LED_THT:LED_D4.0mm, F.Cu at (209.0, 53.0)
- added E57: Electrode out, Connector_Wire:SolderWirePad_1x01_Drill2.5mm, F.Cu at (40.1, 173.5)
- added E58: Electrode out, Connector_Wire:SolderWirePad_1x01_Drill2.5mm, F.Cu at (81.1, 161.5)
- added E59: Electrode out, Connector_Wire:SolderWirePad_1x01_Drill2.5mm, F.Cu at (63.1, 171.5)
- added HV1: G40, HV_source:G40, F.Cu at (72.0, 112.0)
- added HV2: 15A, HV_source:15A, F.Cu at (117.0, 71.0)
- added J1: Low voltage in, Connector_PinHeader_2.54mm:PinHeader_2x01_P2.54mm_Vertical, F.Cu at (187.0, 53.0)
- added J10: Gate, Connector_Wire:SolderWirePad_1x01_Drill2.5mm, F.Cu at (51.1, 172.5)
- added J11: LCD2 Vin, Connector_JST:JST_EH_B2B-EH-A_1x02_P2.50mm_Vertical, F.Cu at (219.0, 118.0)
- added J12: LCD2 PWR, Connector_JST:JST_EH_B2B-EH-A_1x02_P2.50mm_Vertical, F.Cu at (243.0, 118.0)
- added J13: LCD1 V/I measures, Connector_JST:JST_EH_B3B-EH-A_1x03_P2.50mm_Vertical, F.Cu at (229.0, 118.0)
- added J14: LCD1 PWR, Connector_JST:JST_EH_B2B-EH-A_1x02_P2.50mm_Vertical, F.Cu at (254.0, 118.0)
- added J4: Electrode in, Connector_Wire:SolderWirePad_1x01_Drill2.5mm, F.Cu at (69.1, 162.5)
- added J5: Electrode out, Connector_Wire:SolderWirePad_1x01_Drill2.5mm, F.Cu at (32.0, 145.0)
- added J6: HV out, Connector_Wire:SolderWirePad_1x01_Drill2.5mm, F.Cu at (91.1, 160.5)
- added J7: HV out, Connector_Wire:SolderWirePad_1x01_Drill2.5mm, F.Cu at (51.1, 162.5)
- added J8: HV out, Connector_Wire:SolderWirePad_1x01_Drill2.5mm, F.Cu at (59.1, 161.5)
- added POT1: 10M, Potentiometer_THT:Potentiometer_Bourns_3386C_Horizontal, F.Cu at (27.6, 83.6)
- added POT2: 50K, Potentiometer_THT:Potentiometer_Bourns_3386C_Horizontal, F.Cu at (202.0, 145.0)
- added PS1: RHV2-1212S/R20, Isolated_converters:R8, F.Cu at (160.0, 142.0)
- added PS2: RHV2-1212S/R20, Isolated_converters:R20, F.Cu at (185.0, 106.0)
- added Q1: ZVN2110A, Transistors:S8050, F.Cu at (118.0, 8.31)
- added Q2: S8050, Transistors:S8050, F.Cu at (108.0, 106.0)
- added R1: 5K, Resistor_SMD:R_0805_2012Metric_Pad1.15x1.40mm_HandSolder, F.Cu at (134.0, 14.5)
- added R2: 50R, Resistor_SMD:R_0805_2012Metric_Pad1.15x1.40mm_HandSolder, F.Cu at (122.0, 31.0)
- added R3: 1K, Resistor_SMD:R_1206_3216Metric, F.Cu at (138.0, 118.6)
- added R4: 20K, Resistor_SMD:R_0805_2012Metric, F.Cu at (133.0, 120.0)
- added R5: 3.3M, Resistor_SMD:R_0805_2012Metric, F.Cu at (184.0, 68.0)
- added R55: 500K, Resistor_THT:R_Axial_DIN0204_L3.6mm_D1.6mm_P7.62mm_Horizontal, F.Cu at (135.0, 143.0)
- added R56: 1.5M, Resistor_SMD:R_1206_3216Metric, F.Cu at (31.3, 108.2)
- added R57: 1.5M, Resistor_SMD:R_1206_3216Metric, F.Cu at (30.1, 99.0)
- added R58: 1M, Resistor_SMD:R_1206_3216Metric, F.Cu at (213.0, 141.0)
- added R59: 10M, Resistor_SMD:R_1206_3216Metric, F.Cu at (32.3, 113.6)
- added R6: 1M, Resistor_SMD:R_0805_2012Metric, F.Cu at (184.0, 73.0)
- added R64: 100R, Resistor_SMD:R_0805_2012Metric, F.Cu at (244.0, 85.0)
- added R65: 100R, Resistor_SMD:R_0805_2012Metric, F.Cu at (250.0, 55.0)
- added R66: R_LED, Resistor_SMD:R_0805_2012Metric, F.Cu at (201.0, 53.0)
- added SW1: EN switch, Connector_PinHeader_2.54mm:PinHeader_2x01_P2.54mm_Vertical, F.Cu at (213.0, 136.0)
- added SW2: HV1 Switch, Connector_PinHeader_2.54mm:PinHeader_2x01_P2.54mm_Vertical, F.Cu at (213.0, 102.0)
- added SW3: PWR switch, Connector_PinHeader_2.54mm:PinHeader_2x01_P2.54mm_Vertical, F.Cu at (193.5, 53.0)
- added U1: 6N136S, Package_DIP:DIP-8_W10.16mm_LongPads, F.Cu at (115.0, 15.0)
- added U2: mEZD41501A-X, Connector_JST:JST_EH_B6B-EH-A_1x06_P2.50mm_Vertical, F.Cu at (150.5, 112.0)
- added U3: LM358, Package_DIP:DIP-8_W10.16mm_LongPads, F.Cu at (117.0, 106.0)
- added U4: CNY17-1, Package_DIP:DIP-6_W7.62mm, F.Cu at (151.0, 122.5)
- added U5: Lolin32, Dev_boards:Lolin32, F.Cu at (228.0, 73.0)
- added U6: LM358P, Package_DIP:DIP-8_W10.16mm_LongPads, F.Cu at (190.0, 67.0)
Other:
- board size 100 x 100 mm -> 250 x 100 mm
- board text added: "GATE PULSER"

Commit message: Components in place
Parts:
- R7: renamed from R2; footprint Resistor_SMD:R_0805_2012Metric_Pad1.15x1.40mm_HandSolder -> Resistor_SMD:R_1206_3216Metric
- moved R6 140.0 mm to (61.0, 134.0), turned to 90 degrees
- moved C7 137.2 mm to (61.0, 129.0), turned to 90 degrees
- moved C6 137.0 mm to (66.0, 140.0), turned to 270 degrees
- moved Q1 135.3 mm to (55.0, 128.0)
- moved U1 127.1 mm to (76.2, 136.0), turned to 180 degrees
- moved C5 120.3 mm to (56.0, 103.0), turned to 270 degrees
- moved J3 113.9 mm to (26.0, 67.0), turned to 270 degrees
- moved R7 111.0 mm to (57.0, 121.0), turned to 180 degrees
- moved R4 96.1 mm to (39.0, 147.0)
- moved J4 91.0 mm to (26.0, 75.0), turned to 270 degrees
- moved J1 90.4 mm to (26.0, 83.0), turned to 270 degrees
- moved E2 79.6 mm to (26.0, 104.0), turned to 270 degrees
- moved C3 78.1 mm to (38.0, 140.0)
- moved J7 65.5 mm to (26.0, 112.0), turned to 270 degrees
- moved E3 63.5 mm to (26.0, 120.0), turned to 270 degrees
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- renumbered E57 to E1, E58 to E2, E59 to E3, J4 to J1, J13 to J10, J14 to J11, J5 to J2, J6 to J3, J7 to J4, J8 to J5, J1 to J6, J10 to J7, J11 to J8, J12 to J9, R56 to R1, R64 to R10, R65 to R11, R66 to R12, R5 to R13, R6 to R14, R57 to R2, R59 to R3, R55 to R4, R58 to R5, R1 to R6, R3 to R8, R4 to R9
Other:
- board text removed: "GATE PULSER"

Commit message: HV design finished
Parts:
- removed E3: Electrode out, Connector_Wire:SolderWirePad_1x01_Drill2.5mm
- added C11: 100nF, Capacitor_SMD:C_0805_2012Metric, F.Cu at (206.0, 74.0)
- added D2: Protection, Diode_THT:D_T-1_P5.08mm_Horizontal, F.Cu at (171.0, 36.0)
- added F1: Fuse, Fuse:Fuse_1206_3216Metric, F.Cu at (167.0, 36.0)
- added J8: Ap Grid, Connector_Wire:SolderWirePad_1x01_Drill1.5mm, F.Cu at (120.0, 48.0)
- added JP1: Jumper, Connector_PinHeader_1.00mm:PinHeader_1x02_P1.00mm_Horizontal, F.Cu at (232.0, 66.0)
- added OPTO2: CNY65AYST, OptoDevice:CNY65AYST, F.Cu at (162.0, 149.8)
- C5: footprint Capacitor_THT:CP_Radial_D18.0mm_P7.50mm -> Capacitor_THT:CP_Radial_D12.5mm_P5.00mm
- E1: value Electrode out -> Mid electrode1; footprint Connector_Wire:SolderWirePad_1x01_Drill2.5mm -> Connector_Wire:SolderWirePad_1x01_Drill1.5mm
- E2: value Electrode out -> Mid electrode2; footprint Connector_Wire:SolderWirePad_1x01_Drill2.5mm -> Connector_Wire:SolderWirePad_1x01_Drill1.5mm
- J1, J2, J3, J4, J7: footprint Connector_Wire:SolderWirePad_1x01_Drill2.5mm -> Connector_Wire:SolderWirePad_1x01_Drill1.5mm
- J5: value HV out -> Last Electrode; footprint Connector_Wire:SolderWirePad_1x01_Drill2.5mm -> Connector_Wire:SolderWirePad_1x01_Drill1.5mm
- J6: value Low voltage in -> 12V in
- POT1: footprint Potentiometer_THT:Potentiometer_Bourns_3386C_Horizontal -> Potentiometer_THT:Potentiometer_Omeg_PC16BU_Vertical
- POT2: footprint Potentiometer_THT:Potentiometer_Bourns_3386C_Horizontal -> Potentiometer_THT:Potentiometer_Piher_T-16H_Single_Horizontal
- Q2: value S8050 -> ZTX1053A
- R4: renamed from R5; footprint Resistor_SMD:R_1206_3216Metric -> Resistor_SMD:R_0805_2012Metric
- U4: value CNY17-1 -> MC78M15ACTG; footprint Package_DIP:DIP-6_W7.62mm -> Package_TO_SOT_THT:TO-262-3_Vertical
- moved J5 154.3 mm to (131.0, 31.0), turned to 90 degrees
- moved J12 149.9 mm to (108.0, 152.0)
- moved R1 138.4 mm to (123.0, 37.0), turned to 90 degrees
- moved C3 127.0 mm to (115.0, 39.0), turned to 90 degrees
- moved J11 117.0 mm to (117.0, 152.0)
- moved J2 112.4 mm to (105.0, 48.0), turned to 0 degrees
- moved J7 108.0 mm to (113.0, 48.0), turned to 0 degrees
- moved E1 102.7 mm to (79.0, 48.0), turned to 0 degrees
- moved C2 102.6 mm to (97.0, 39.0), turned to 90 degrees
- moved U4 92.7 mm to (224.1, 67.0)
- moved R5 90.6 mm to (100.0, 48.0), turned to 180 degrees
- moved C7 89.6 mm to (113.0, 56.0)
- moved R6 89.6 mm to (113.0, 61.0)
- moved C6 89.6 mm to (115.0, 65.0), turned to 180 degrees
- moved OPTO1 89.3 mm to (126.2, 62.0)
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- renumbered J9 to J10, J10 to J11, J11 to J12, J8 to J9, U1 to OPTO1, R4 to R1, R1 to R2, R2 to R3, R3 to R5, R9 to R8, R8 to R9, U2 to U1, U3 to U2, U5 to U3, U6 to U5
Connections:
- C10 pad 2: LAST_ELECTRODE -> GND
- C8 pad 2: GATE_OUT -> GNDB
- C9 pad 2: GATE_OUT -> GNDB
- D1 pad 1: LAST_ELECTRODE -> GND
- E1 pad 1: /Aperture_Grid -> /Middle_electrode1
- E2 pad 1: /Middle_electrode1 -> /Middle_electrode2
- HV2 pad 1: LAST_ELECTRODE -> GND
- J10 pad 2: LAST_ELECTRODE -> GND
- J11 pad 3: GATE_OUT -> GNDB
- J12 pad 2: GATE_OUT -> GNDB
- J6 pad 1: Net-(J6-Pad1) -> Net-(F1-Pad1)
- J6 pad 2: LAST_ELECTRODE -> GND
- J9 pad 2: LAST_ELECTRODE -> GND
- OPTO1 pad 3: LAST_ELECTRODE -> GND
- PS1 pad 1: LAST_ELECTRODE -> +12V
- PS1 pad 2: +12V -> GND
- PS2 pad 1: LAST_ELECTRODE -> +12V
- PS2 pad 2: +12V -> GND
- PS2 pad 3: GATE_OUT -> GNDB
- R14 pad 2: LAST_ELECTRODE -> GND
- R4 pad 1: LAST_ELECTRODE -> GND
- R8 pad 1: Net-(R8-Pad1) -> Net-(OPTO2-Pad3)
- R9 pad 1: Net-(R8-Pad1) -> GNDB
- R9 pad 2: +15V -> Net-(OPTO2-Pad3)
- SW3 pad 2: Net-(J6-Pad1) -> Net-(D2-Pad1)
- U1 pad 3: GATE_OUT -> GNDB
- U1 pad 4: GATE_OUT -> GNDB
- U2 pad 4: GATE_OUT -> GNDB
- U2 pad 5: GATE_OUT -> GNDB
- U3 pad 15: (no net) -> +5V
- U3 pad 16: LAST_ELECTRODE -> GND
- U3 pad 17: LAST_ELECTRODE -> GND
- U3 pad 23: LAST_ELECTRODE -> GND
- U3 pad 24: LAST_ELECTRODE -> GND
- U3 pad 34: LAST_ELECTRODE -> GND
- U4 pad 1: PWM -> Net-(JP1-Pad2)
- U4 pad 2: LAST_ELECTRODE -> GND
- U4 pad 3: (no net) -> +5V
- U5 pad 4: LAST_ELECTRODE -> GND
- U5 pad 6: LAST_ELECTRODE -> GND
Routing:
- net EOUT: track 0.00 -> 93.7 mm, vias 0 -> 1
- net ALIMHV1+: track 0.00 -> 67.1 mm
- net Net-(HV2-Pad5): track 0.00 -> 49.0 mm
- net Net-(HV2-Pad6): track 0.00 -> 41.8 mm
- net +15V: track 0.00 -> 37.8 mm, vias 0 -> 22
- net Net-(HV2-Pad7): track 0.00 -> 34.7 mm
- net GATE_IN+: track 0.00 -> 33.7 mm
- net Net-(C9-Pad1): track 0.00 -> 31.7 mm
- net PWM: track 0.00 -> 30.6 mm
- net GATE_IN-: track 0.00 -> 25.3 mm
- net ALIMHV1-: track 0.00 -> 22.9 mm
- net /Middle_electrode1: track 0.00 -> 20.8 mm
- net Net-(C7-Pad1): track 0.00 -> 20.3 mm
- net /Aperture_Grid: track 0.00 -> 19.3 mm
- net Net-(OPTO2-Pad3): track 0.00 -> 19.2 mm
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- added copper zone on F.Cu, net +12V
- added copper zone on F.Cu, net +15V
- added copper zone on B.Cu, net GATE_OUT
- added copper zone on F.Cu, net GATE_OUT
- added copper zone on B.Cu, net GND
- added copper zone on B.Cu, net GNDB
- added copper zone on F.Cu, net LAST_ELECTRODE
Other:
- board size 250 x 100 mm -> 193 x 130 mm
- board text added: "LCD1"
- board text added: "LCD2"

Commit message: Improve PCBs
Parts:
- removed OPTO1: 6N136S, Package_DIP:DIP-8_W10.16mm_LongPads
- added C12: 0.33uF Tant., Capacitor_Tantalum_SMD:CP_EIA-3528-21_Kemet-B_Pad1.50x2.35mm_HandSolder, F.Cu at (231.0, 73.0)
- added TP10: TestPoint, TestPoint:TestPoint_Keystone_5000-5004_Miniature, F.Cu at (116.0, 119.0)
- added TP11: TestPoint, TestPoint:TestPoint_Keystone_5000-5004_Miniature, F.Cu at (117.0, 145.0)
- added TP12: TestPoint, TestPoint:TestPoint_Keystone_5000-5004_Miniature, F.Cu at (106.0, 145.0)
- added TP13: TestPoint, TestPoint:TestPoint_Keystone_5000-5004_Miniature, F.Cu at (182.0, 74.0)
- added TP14: TestPoint, TestPoint:TestPoint_Keystone_5000-5004_Miniature, F.Cu at (190.0, 69.0)
- added TP15: TestPoint, TestPoint:TestPoint_Keystone_5000-5004_Miniature, F.Cu at (200.0, 66.0)
- added TP2: TestPoint, TestPoint:TestPoint_Keystone_5000-5004_Miniature, F.Cu at (113.0, 53.0)
- added TP4: TestPoint, TestPoint:TestPoint_Keystone_5000-5004_Miniature, F.Cu at (89.0, 67.0)
- added TP5: TestPoint, TestPoint:TestPoint_Keystone_5000-5004_Miniature, F.Cu at (128.0, 133.0)
- added TP6: TestPoint, TestPoint:TestPoint_Keystone_5000-5004_Miniature, F.Cu at (96.0, 72.0)
- added TP7: TestPoint, TestPoint:TestPoint_Keystone_5000-5004_Miniature, F.Cu at (130.0, 152.0)
- added TP8: TestPoint, TestPoint:TestPoint_Keystone_5000-5004_Miniature, F.Cu at (87.0, 45.0)
- added TP9: TestPoint, TestPoint:TestPoint_Keystone_5000-5004_Miniature, F.Cu at (111.0, 145.0)
- added U6: 6N137A, Package_DIP:DIP-8_W7.62mm_Socket, F.Cu at (124.5, 62.5)
- Q1, Q2: footprint Transistors:S8050 -> Package_TO_SOT_THT:TO-220-3_Vertical
- U2, U5: footprint Package_DIP:DIP-8_W10.16mm_LongPads -> Package_DIP:DIP-8_W7.62mm_Socket
- moved C9 3.61 mm to (113.0, 139.0), turned to 0 degrees
- moved J10 2.83 mm to (243.0, 100.0)
- moved C8 2.50 mm to (126.8, 125.9)
- moved Q2 1.84 mm to (110.0, 127.5)
- moved C6 1.00 mm to (116.0, 65.0)
- moved C7 1.00 mm to (113.0, 57.0)
- moved J8 1.00 mm to (121.0, 48.0)
Routing:
- net GATE_OUT: track 0.00 -> 9.77 mm
- net Net-(Q2-Pad2): track 7.37 -> 6.25 mm
- net Net-(C9-Pad1): track 31.7 -> 32.7 mm
- net +12VA: track 16.3 -> 17.3 mm
Other:
- outline, holes or cut-outs redrawn
- board text added: "E B C"
- board text added: "QUESTIONS : - GND/VCC planes coupés - Comment relier HV GND et HV2? - Pistes arondies pour HV? (dans le diviseur) - Tailles des packages (OPTO2) isolation : (DC/DC : 20kV, opto : 13kV) - Isolation LCD - PCB Gate"

Commit message: Improve PCBs
Parts:
- moved Q1 5.44 mm to (99.5, 72.0)
- moved TP6 2.00 mm to (94.0, 72.0)
Routing:
- net Net-(C7-Pad1): track 20.4 -> 23.3 mm
Changed lines of the file:
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@@
     (thickness 1.6)
     (drawings 16)
-    (tracks 172)
+    (tracks 171)
     (zones 0)
     (modules 75)
@@
   )
   (module Package_TO_SOT_THT:TO-220-3_Vertical (layer F.Cu)
-    (at 104 69)
+    (at 99.46 72)
     (descr "TO-220-3, Vertical, RM 2.54mm, see https://www.vishay.com/docs/66542/to-220-1.pdf")
     (tags "TO-220-3 Vertical RM 2.54mm")
@@
   )
   (module TestPoint:TestPoint_Keystone_5000-5004_Miniature (layer F.Cu)
-    (at 96 72)
+    (at 94 72)
     (descr "Keystone Miniature THM Test Point 5000-5004, http://www.keyelco.com/product-pdf.cfm?p=1309")
     (tags "Through Hole Mount Test Points")
@@
   (segment (start 85 63) (end 97 63) (width 1) (layer F.Cu) (net 8))
   (segment (start 77 55) (end 85 63) (width 1) (layer F.Cu) (net 8))
-  (segment (start 102.73 67.57) (end 102.73 69.69) (width 1) (layer F.Cu) (net 8))
-  (segment (start 102.73 66.53) (end 102.73 67.57) (width 1) (layer F.Cu) (net 8))
-  (segment (start 99.2 63) (end 102.73 66.53) (width 1) (layer F.Cu) (net 8))
-  (segment (start 97 63) (end 99.2 63) (width 1) (layer F.Cu) (net 8))
+  (segment (start 97 63) (end 97 67) (width 1) (layer F.Cu) (net 8))
+  (segment (start 99.46 69.46) (end 99.46 72) (width 1) (layer F.Cu) (net 8))
+  (segment (start 97 67) (end 99.46 69.46) (width 1) (layer F.Cu) (net 8))
   (via (at 70 68) (size 0.8) (drill 0.4) (layers F.Cu B.Cu) (net 9))
   (via (at 106 75) (size 0.8) (drill 0.4) (layers F.Cu B.Cu) (net 9))
@@
   (segment (start 116.88 62.5) (end 113.475 62.5) (width 1) (layer F.Cu) (net 10))
   (segment (start 112.3 59.975) (end 113 59.975) (width 1) (layer F.Cu) (net 11))
-  (segment (start 111.595 59.975) (end 112.3 59.975) (width 1) (layer F.Cu) (net 11))
-  (segment (start 104 67.57) (end 111.595 59.975) (width 1) (layer F.Cu) (net 11))
-  (segment (start 104 69.69) (end 104 67.57) (width 1) (layer F.Cu) (net 11))
+  (segment (start 112.025 59.975) (end 112.3 59.975) (width 1) (layer F.Cu) (net 11))
+  (segment (start 102 70) (end 112.025 59.975) (width 1) (layer F.Cu) (net 11))
+  (segment (start 102 72) (end 102 70) (width 1) (layer F.Cu) (net 11))
+  (segment (start 113 59.975) (end 113 57.9375) (width 1) (layer F.Cu) (net 11))
   (segment (start 116.3625 57.9375) (end 116.88 57.42) (width 1) (layer F.Cu) (net 11))
   (segment (start 113 57.9375) (end 116.3625 57.9375) (width 1) (layer F.Cu) (net 11))
-  (segment (start 113 57.9375) (end 113 59.975) (width 1) (layer F.Cu) (net 11))
   (via (at 127 143) (size 0.8) (drill 0.4) (layers F.Cu B.Cu) (net 12))
   (segment (start 127 143) (end 129 141) (width 0.7) (layer B.Cu) (net 12))

Commit message: Alim&control update
Parts:
- removed D2: Protection, Diode_THT:D_T-1_P5.08mm_Horizontal
- removed F1: Fuse, Fuse:Fuse_1206_3216Metric
- removed POT2: 50K, Potentiometer_THT:Potentiometer_Piher_T-16H_Single_Horizontal
- removed TP10, TP11, TP9: TestPoint, TestPoint:TestPoint_Keystone_5000-5004_Miniature
- removed the TP2 at (113.0, 53.0)
- removed the TP5 at (128.0, 133.0)
- removed the TP6 at (94.0, 72.0)
- removed the TP7 at (130.0, 152.0)
- added C13: 2,2uF, Capacitor_SMD:C_0805_2012Metric_Pad1.15x1.40mm_HandSolder, F.Cu at (180.0, 79.0)
- added POT3: 50K, Potentiometer_THT:Potentiometer_Alps_RK097_Single_Horizontal, F.Cu at (241.0, 104.5)
- added POT4: 50K, Potentiometer_THT:Potentiometer_Alps_RK097_Single_Horizontal, F.Cu at (241.0, 136.5)
- added Q3: SSM3J340R, Package_TO_SOT_SMD:SOT-23_Handsoldering, F.Cu at (166.9, 36.4)
- added Q4: ZTX1053A, Package_TO_SOT_SMD:SOT-23_Handsoldering, F.Cu at (185.0, 78.0)
- added R15: 20K, Resistor_SMD:R_0805_2012Metric, F.Cu at (180.0, 74.0)
- added R16: 20K, Resistor_SMD:R_0805_2012Metric, F.Cu at (181.0, 82.0)
- E1, E2, J1, J2, J3, J4, J5, J8: footprint Connector_Wire:SolderWirePad_1x01_Drill1.5mm -> Connector:conn_HV_JACK_PB1021
- J6: renamed from J7; footprint Connector_Wire:SolderWirePad_1x01_Drill1.5mm -> Connector:conn_HV_JACK_PB1021
- POT1: footprint Potentiometer_THT:Potentiometer_Omeg_PC16BU_Vertical -> Potentiometer_THT:Potentiometer_Vishay_148-149_Single_Vertical
- moved TP2 75.5 mm to (90.9, -8.50)
- moved POT1 43.0 mm to (111.5, 38.0)
- moved R1 41.7 mm to (93.0, 66.0), turned to 270 degrees
- moved J5 41.7 mm to (95.0, 52.0), turned to 0 degrees
- moved J4 38.1 mm to (44.0, 86.0), turned to 180 degrees
- moved C3 37.5 mm to (87.0, 64.0), turned to 270 degrees
- moved C4 33.8 mm to (44.0, 72.0), turned to 0 degrees
- moved J8 33.2 mm to (88.0, 52.0)
- moved C2 32.0 mm to (77.0, 64.0), turned to 270 degrees
- moved C12 30.7 mm to (177.0, 64.0)
- moved J1 30.3 mm to (102.0, 52.0), turned to 0 degrees
- moved R13 27.9 mm to (162.2, 65.0)
- moved R14 27.9 mm to (162.2, 70.0)
- moved TP6 27.9 mm to (156.0, 64.0)
- moved TP7 27.9 mm to (164.0, 59.0)
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- renumbered C12 to C10, C10 to C11, C11 to C12, J6 to J7, OPTO2 to OPTO1, TP4 to TP2, TP8 to TP4, TP12 to TP5, TP13 to TP6, TP14 to TP7, TP15 to TP8, U6 to U1, U1 to U2, U2 to U3, U3 to U4, U4 to U5, U5 to U6
Connections:
- HV2 pad 5: Net-(HV2-Pad5) -> (no net)
- HV2 pad 6: Net-(HV2-Pad6) -> ADJ_HV2
- HV2 pad 7: Net-(HV2-Pad7) -> (no net)
- JP1 pad 1: +12V -> +5V
- U4 pad 15: +5V -> Net-(JP1-Pad2)
- U4 pad 5: (no net) -> ADJ_HV2_PWM
- U4 pad 6: (no net) -> ADC1
- U4 pad 7: (no net) -> ADC2
- U5 pad 1: Net-(JP1-Pad2) -> +12V
Routing:
- net /Middle_electrode1: track 20.8 -> 104.3 mm
- net GATE_IN-: track 25.3 -> 91.9 mm
- net Net-(HV2-Pad5): track 49.0 -> 0.00 mm
- net Net-(HV2-Pad6): track 41.8 -> 0.00 mm
- net Net-(HV2-Pad7): track 34.7 -> 0.00 mm
- net PWM: track 30.6 -> 0.00 mm
- net LAST_ELECTRODE: track 0.00 -> 27.4 mm
- net EOUT: track 93.7 -> 72.7 mm, vias 1 -> 0
- net GATE_OUT: track 9.77 -> 29.6 mm, vias 9 -> 2
- net TRI-STATE: track 7.00 -> 26.1 mm
- net Net-(HV2-Pad4): track 14.2 -> 0.00 mm
- net LCD2_MEASURE: track 14.0 -> 0.00 mm
- net /Middle_electrode2: track 17.0 -> 30.1 mm
- net DRIFT_TUBE: track 3.60 -> 14.7 mm
- net GND: track 3.83 -> 14.3 mm
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- added copper zone on F.Cu, net COUNTER_ELECTRODE
Other:
- board size 193 x 130 mm -> 208 x 130 mm
