File: PCB/Divider/Complete_divider/VoltageMeasurements.sch (KiCad schematic (older format))
At the start: 8 parts, among them J10 LCD2 PWR, J11 LCD1 V/I measures, J12 LCD1 PWR, J9 LCD2 Vin, U5 LM358P

Commit message: Improve PCBs
Parts:
- added TP13, TP14, TP15: TestPoint, TestPoint:TestPoint_Keystone_5000-5004_Miniature, symbol Connector:TestPoint
- U5: footprint Package_DIP:DIP-8_W10.16mm_LongPads -> Package_DIP:DIP-8_W7.62mm_Socket
Connections:
- net EOUT: now also TP13.1
- net EOUTPIN: now also TP15.1
- net at R13.2, R14.1, U5.3 (+): now also TP14.1
Changed lines of the file:
@@
 F 0 "U5" H 7150 3517 50  0000 C CNN
 F 1 "LM358P" H 7150 3426 50  0000 C CNN
-F 2 "Package_DIP:DIP-8_W10.16mm_LongPads" H 7150 3150 50  0001 C CNN
+F 2 "Package_DIP:DIP-8_W7.62mm_Socket" H 7150 3150 50  0001 C CNN
 F 3 "http://www.ti.com/lit/ds/symlink/lm2904-n.pdf" H 7150 3150 50  0001 C CNN
 	1    7150 3150
@@
 F 0 "U5" H 8800 3517 50  0000 C CNN
 F 1 "LM358P" H 8800 3426 50  0000 C CNN
-F 2 "Package_DIP:DIP-8_W10.16mm_LongPads" H 8800 3150 50  0001 C CNN
+F 2 "Package_DIP:DIP-8_W7.62mm_Socket" H 8800 3150 50  0001 C CNN
 F 3 "http://www.ti.com/lit/ds/symlink/lm2904-n.pdf" H 8800 3150 50  0001 C CNN
 	2    8800 3150
@@
 F 0 "U5" H 7958 4396 50  0000 L CNN
 F 1 "LM358P" H 7958 4305 50  0000 L CNN
-F 2 "Package_DIP:DIP-8_W10.16mm_LongPads" H 8000 4350 50  0001 C CNN
+F 2 "Package_DIP:DIP-8_W7.62mm_Socket" H 8000 4350 50  0001 C CNN
 F 3 "http://www.ti.com/lit/ds/symlink/lm2904-n.pdf" H 8000 4350 50  0001 C CNN
 	3    8000 4350
@@
 	1    0    0    -1
 $EndComp
+$Comp
+L Connector:TestPoint TP13
+U 1 1 5EFC7F61
+P 6700 2500
+F 0 "TP13" H 6758 2572 50  0000 L CNN
+F 1 "TestPoint" H 6758 2527 50  0001 L CNN
+F 2 "TestPoint:TestPoint_Keystone_5000-5004_Miniature" H 6900 2500 50  0001 C CNN
+F 3 "~" H 6900 2500 50  0001 C CNN
+	1    6700 2500
+	1    0    0    -1
+$EndComp
+Wire Wire Line
+	6700 2500 6700 2550
+Connection ~ 6700 2550
+$Comp
+L Connector:TestPoint TP14
+U 1 1 5EFC8FB3
+P 6550 3050
+F 0 "TP14" V 6653 3122 50  0000 C CNN
+F 1 "TestPoint" H 6608 3077 50  0001 L CNN
+F 2 "TestPoint:TestPoint_Keystone_5000-5004_Miniature" H 6750 3050 50  0001 C CNN
+F 3 "~" H 6750 3050 50  0001 C CNN
+	1    6550 3050
+	0    -1   -1   0
+$EndComp
+Wire Wire Line
+	6550 3050 6700 3050
+$Comp
+L Connector:TestPoint TP15
+U 1 1 5EFCA1A9
+P 7450 3050
+F 0 "TP15" H 7508 3122 50  0000 L CNN
+F 1 "TestPoint" H 7508 3077 50  0001 L CNN
+F 2 "TestPoint:TestPoint_Keystone_5000-5004_Miniature" H 7650 3050 50  0001 C CNN
+F 3 "~" H 7650 3050 50  0001 C CNN
+	1    7450 3050
+	1    0    0    -1
+$EndComp
+Wire Wire Line
+	7450 3050 7450 3150
 $EndSCHEMATC

Commit message: Alim&control update
Parts:
- renumbered C11 to C12, TP14 to TP10, TP15 to TP11, TP13 to TP9, U5 to U6
Changed lines of the file:
@@
 AR Path="/5E63F098/5EDCBED7" Ref="#PWR?"  Part="1"
 AR Path="/5E63F098/5EDBC18D/5EDCBED7" Ref="#PWR?"  Part="1"
-AR Path="/5EDBC18D/5EDCBED7" Ref="#PWR043"  Part="1"
-F 0 "#PWR043" H 6700 3350 50  0001 C CNN
+AR Path="/5EDBC18D/5EDCBED7" Ref="#PWR044"  Part="1"
+F 0 "#PWR044" H 6700 3350 50  0001 C CNN
 F 1 "GND" H 6705 3427 50  0000 C CNN
 F 2 "" H 6700 3600 50  0001 C CNN
@@
 AR Path="/5E63F098/5EDCBEE3" Ref="U?"  Part="1"
 AR Path="/5E63F098/5EDBC18D/5EDCBEE3" Ref="U?"  Part="1"
-AR Path="/5EDBC18D/5EDCBEE3" Ref="U5"  Part="1"
-F 0 "U5" H 7150 3517 50  0000 C CNN
+AR Path="/5EDBC18D/5EDCBEE3" Ref="U6"  Part="1"
+F 0 "U6" H 7150 3517 50  0000 C CNN
 F 1 "LM358P" H 7150 3426 50  0000 C CNN
 F 2 "Package_DIP:DIP-8_W7.62mm_Socket" H 7150 3150 50  0001 C CNN
@@
 AR Path="/5E63F098/5EDCBEEE" Ref="U?"  Part="2"
 AR Path="/5E63F098/5EDBC18D/5EDCBEEE" Ref="U?"  Part="2"
-AR Path="/5EDBC18D/5EDCBEEE" Ref="U5"  Part="2"
-F 0 "U5" H 8800 3517 50  0000 C CNN
+AR Path="/5EDBC18D/5EDCBEEE" Ref="U6"  Part="2"
+F 0 "U6" H 8800 3517 50  0000 C CNN
 F 1 "LM358P" H 8800 3426 50  0000 C CNN
 F 2 "Package_DIP:DIP-8_W7.62mm_Socket" H 8800 3150 50  0001 C CNN
@@
 AR Path="/5E63F098/5EDCBEF7" Ref="#PWR?"  Part="1"
 AR Path="/5E63F098/5EDBC18D/5EDCBEF7" Ref="#PWR?"  Part="1"
-AR Path="/5EDBC18D/5EDCBEF7" Ref="#PWR042"  Part="1"
-F 0 "#PWR042" H 8450 3050 50  0001 C CNN
+AR Path="/5EDBC18D/5EDCBEF7" Ref="#PWR043"  Part="1"
+F 0 "#PWR043" H 8450 3050 50  0001 C CNN
 F 1 "GND" H 8455 3127 50  0000 C CNN
 F 2 "" H 8450 3300 50  0001 C CNN
@@
 	8450 3250 8500 3250
 $Comp
-L Amplifier_Operational:LM358 U5
+L Amplifier_Operational:LM358 U6
 U 3 1 5EDCFF75
 P 8000 4350
-F 0 "U5" H 7958 4396 50  0000 L CNN
+F 0 "U6" H 7958 4396 50  0000 L CNN
 F 1 "LM358P" H 7958 4305 50  0000 L CNN
 F 2 "Package_DIP:DIP-8_W7.62mm_Socket" H 8000 4350 50  0001 C CNN
@@
 $EndComp
 $Comp
-L power:+12V #PWR045
+L power:+12V #PWR046
 U 1 1 5EDD48A6
 P 7900 4000
-F 0 "#PWR045" H 7900 3850 50  0001 C CNN
+F 0 "#PWR046" H 7900 3850 50  0001 C CNN
 F 1 "+12V" H 7915 4173 50  0000 C CNN
 F 2 "" H 7900 4000 50  0001 C CNN
@@
 AR Path="/5E63F098/5EDD5377" Ref="#PWR?"  Part="1"
 AR Path="/5E63F098/5EDBC18D/5EDD5377" Ref="#PWR?"  Part="1"
-AR Path="/5EDBC18D/5EDD5377" Ref="#PWR048"  Part="1"
-F 0 "#PWR048" H 7900 4450 50  0001 C CNN
+AR Path="/5EDBC18D/5EDD5377" Ref="#PWR049"  Part="1"
+F 0 "#PWR049" H 7900 4450 50  0001 C CNN
 F 1 "GND" H 7905 4527 50  0000 C CNN
 F 2 "" H 7900 4700 50  0001 C CNN
@@
 AR Path="/5E63F098/5EDE3C96" Ref="#PWR?"  Part="1"
 AR Path="/5E63F098/5EDBC18D/5EDE3C96" Ref="#PWR?"  Part="1"
-AR Path="/5EDBC18D/5EDE3C96" Ref="#PWR041"  Part="1"
-F 0 "#PWR041" H 4850 3000 50  0001 C CNN
+AR Path="/5EDBC18D/5EDE3C96" Ref="#PWR042"  Part="1"
+F 0 "#PWR042" H 4850 3000 50  0001 C CNN
 F 1 "GND" H 4855 3077 50  0000 C CNN
 F 2 "" H 4850 3250 50  0001 C CNN
@@
 	4700 3100 4850 3100
 $Comp
-L power:+12V #PWR039
+L power:+12V #PWR040
 U 1 1 5EDE2C72
 P 4850 3050
-F 0 "#PWR039" H 4850 2900 50  0001 C CNN
+F 0 "#PWR040" H 4850 2900 50  0001 C CNN
 F 1 "+12V" H 4865 3223 50  0000 C CNN
 F 2 "" H 4850 3050 50  0001 C CNN
@@
 AR Path="/5E63F098/5EDE1095" Ref="#PWR?"  Part="1"
 AR Path="/5E63F098/5EDBC18D/5EDE1095" Ref="#PWR?"  Part="1"
-AR Path="/5EDBC18D/5EDE1095" Ref="#PWR040"  Part="1"
-F 0 "#PWR040" H 3300 3000 50  0001 C CNN
+AR Path="/5EDBC18D/5EDE1095" Ref="#PWR041"  Part="1"
+F 0 "#PWR041" H 3300 3000 50  0001 C CNN
 F 1 "GND" H 3305 3077 50  0000 C CNN
 F 2 "" H 3300 3250 50  0001 C CNN
@@
 1 : I measure \n2 : V measure\n
 $Comp
-L power:+15V #PWR044
+L power:+15V #PWR045
 U 1 1 5F1DF154
 P 4850 3950
-F 0 "#PWR044" H 4850 3800 50  0001 C CNN
+F 0 "#PWR045" H 4850 3800 50  0001 C CNN
 F 1 "+15V" H 4865 4123 50  0000 C CNN
 F 2 "" H 4850 3950 50  0001 C CNN
@@
 $EndComp
 $Comp
-L Device:C_Small C11
+L Device:C_Small C12
 U 1 1 5F7E26A8
 P 7650 4350
-F 0 "C11" H 7559 4304 50  0000 R CNN
+F 0 "C12" H 7559 4304 50  0000 R CNN
 F 1 "100nF" H 7559 4395 50  0000 R CNN
 F 2 "Capacitor_SMD:C_0805_2012Metric" H 7650 4350 50  0001 C CNN
@@
 Connection ~ 7900 4650
 $Comp
-L power:GNDB #PWR046
+L power:GNDB #PWR047
 U 1 1 5F86EA85
 P 3300 4150
-F 0 "#PWR046" H 3300 3900 50  0001 C CNN
+F 0 "#PWR047" H 3300 3900 50  0001 C CNN
 F 1 "GNDB" H 3305 3977 50  0000 C CNN
 F 2 "" H 3300 4150 50  0001 C CNN
@@
 $EndComp
 $Comp
-L power:GNDB #PWR047
+L power:GNDB #PWR048
 U 1 1 5F86F04D
 P 4850 4150
-F 0 "#PWR047" H 4850 3900 50  0001 C CNN
+F 0 "#PWR048" H 4850 3900 50  0001 C CNN
 F 1 "GNDB" H 4855 3977 50  0000 C CNN
 F 2 "" H 4850 4150 50  0001 C CNN
@@
 $EndComp
 $Comp
-L Connector:TestPoint TP13
+L Connector:TestPoint TP9
 U 1 1 5EFC7F61
 P 6700 2500
-F 0 "TP13" H 6758 2572 50  0000 L CNN
+F 0 "TP9" H 6758 2572 50  0000 L CNN
 F 1 "TestPoint" H 6758 2527 50  0001 L CNN
 F 2 "TestPoint:TestPoint_Keystone_5000-5004_Miniature" H 6900 2500 50  0001 C CNN
@@
 Connection ~ 6700 2550
 $Comp
-L Connector:TestPoint TP14
+L Connector:TestPoint TP10
 U 1 1 5EFC8FB3
 P 6550 3050
-F 0 "TP14" V 6653 3122 50  0000 C CNN
+F 0 "TP10" V 6653 3122 50  0000 C CNN
 F 1 "TestPoint" H 6608 3077 50  0001 L CNN
 F 2 "TestPoint:TestPoint_Keystone_5000-5004_Miniature" H 6750 3050 50  0001 C CNN
@@
 	6550 3050 6700 3050
 $Comp
-L Connector:TestPoint TP15
+L Connector:TestPoint TP11
 U 1 1 5EFCA1A9
 P 7450 3050
-F 0 "TP15" H 7508 3122 50  0000 L CNN
+F 0 "TP11" H 7508 3122 50  0000 L CNN
 F 1 "TestPoint" H 7508 3077 50  0001 L CNN
 F 2 "TestPoint:TestPoint_Keystone_5000-5004_Miniature" H 7650 3050 50  0001 C CNN
