File: PCB/Ampli/Ampli_IMS.kicad_pcb (KiCad board)
At the start: 2 copper layers, 44.4 x 28.5 mm, 15 parts, among them J1 5227161-3, J2 5227161-3, J3 Conn_01x03_Male, P1 300K, U1 LMC6082

Commit message: Update
Routing:
- net GND: vias 228 -> 240
Changed lines of the file:
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@@
     (thickness 1.6)
     (drawings 11)
-    (tracks 287)
+    (tracks 299)
     (zones 0)
     (modules 15)
@@
     (32 B.Adhes user)
     (33 F.Adhes user)
-    (34 B.Paste user hide)
+    (34 B.Paste user)
     (35 F.Paste user)
-    (36 B.SilkS user hide)
+    (36 B.SilkS user)
     (37 F.SilkS user)
-    (38 B.Mask user hide)
+    (38 B.Mask user)
     (39 F.Mask user)
     (40 Dwgs.User user)
@@
     (44 Edge.Cuts user)
     (45 Margin user)
-    (46 B.CrtYd user hide)
+    (46 B.CrtYd user)
     (47 F.CrtYd user)
     (48 B.Fab user)
-    (49 F.Fab user hide)
+    (49 F.Fab user)
   )
   (setup
@@
     (mod_text_size 1 1)
     (mod_text_width 0.15)
-    (pad_size 3.5 7)
-    (pad_drill 2.01)
+    (pad_size 1.7 1.95)
+    (pad_drill 0.95)
     (pad_to_mask_clearance 0)
     (aux_axis_origin 0 0)
@@
     (pcbplotparams
       (layerselection 0x010fc_ffffffff)
-      (usegerberextensions false)
+      (usegerberextensions true)
       (usegerberattributes false)
       (usegerberadvancedattributes false)
@@
       (outputformat 1)
       (mirror false)
-      (drillshape 1)
+      (drillshape 0)
       (scaleselection 1)
-      (outputdirectory ""))
+      (outputdirectory "/Users/valentin/Desktop/GERBER_IMS_1/"))
   )
   (net 0 "")
@@
     (descr https://www.amphenolrf.com/media/downloads/1769/132203-12.pdf)
     (tags "SMA THT Female Jack Horizontal")
+    (zone_connect 2)
     (fp_text reference J1 (at -5.2 0) (layer F.SilkS)
       (effects (font (size 1 1) (thickness 0.15)))
@@
     (fp_line (start -3.175 -18) (end 3.175 -18.706) (layer F.Fab) (width 0.1))
     (pad 1 thru_hole circle (at 0 0 90) (size 2.25 2.25) (drill 1.5) (layers *.Cu *.Mask)
-      (net 6 "Net-(C1-Pad2)"))
+      (net 6 "Net-(C1-Pad2)") (zone_connect 2))
     (pad 2 thru_hole circle (at 2.54 2.54 180) (size 2.25 2.25) (drill 1.7) (layers *.Cu *.Mask)
-      (net 1 GND))
+      (net 1 GND) (zone_connect 2))
     (pad 2 thru_hole circle (at 2.54 -2.54 90) (size 2.25 2.25) (drill 1.7) (layers *.Cu *.Mask)
-      (net 1 GND))
+      (net 1 GND) (zone_connect 2))
     (pad 2 thru_hole circle (at -2.54 -2.54 90) (size 2.25 2.25) (drill 1.7) (layers *.Cu *.Mask)
-      (net 1 GND))
+      (net 1 GND) (zone_connect 2))
     (pad 2 thru_hole circle (at -2.54 2.54 90) (size 2.25 2.25) (drill 1.7) (layers *.Cu *.Mask)
-      (net 1 GND))
+      (net 1 GND) (zone_connect 2))
     (model ${KISYS3DMOD}/Connector_Coaxial.3dshapes/SMA_Amphenol_132203-12_Horizontal.wrl
       (at (xyz 0 0 0))
@@
       (net 3 "Net-(D2-Pad1)"))
     (pad 2 thru_hole oval (at 2.5 0 180) (size 1.7 1.95) (drill 0.95) (layers *.Cu *.Mask)
-      (net 1 GND))
+      (net 1 GND) (zone_connect 1))
     (pad 1 thru_hole roundrect (at 0 0 180) (size 1.7 1.95) (drill 0.95) (layers *.Cu *.Mask) (roundrect_rratio 0.147059)
       (net 2 "Net-(D1-Pad2)"))
@@
   (via (at 66 39) (size 0.8) (drill 0.4) (layers F.Cu B.Cu) (net 1))
   (via (at 68 39) (size 0.8) (drill 0.4) (layers F.Cu B.Cu) (net 1))
-  (via (at 56 39) (size 0.8) (drill 0.4) (layers F.Cu B.Cu) (net 1))
   (via (at 58 39) (size 0.8) (drill 0.4) (layers F.Cu B.Cu) (net 1))
   (via (at 54 39) (size 0.8) (drill 0.4) (layers F.Cu B.Cu) (net 1))
@@
   (via (at 44 27) (size 0.8) (drill 0.4) (layers F.Cu B.Cu) (net 1))
   (via (at 48 27) (size 0.8) (drill 0.4) (layers F.Cu B.Cu) (net 1))
-  (via (at 49 31) (size 0.8) (drill 0.4) (layers F.Cu B.Cu) (net 1))
   (via (at 47.5 32.5) (size 0.8) (drill 0.4) (layers F.Cu B.Cu) (net 1))
   (via (at 31.8 34.9) (size 0.5) (drill 0.3) (layers F.Cu B.Cu) (net 1))
@@
   (via (at 34 31) (size 0.8) (drill 0.4) (layers F.Cu B.Cu) (net 1))
   (via (at 44 35) (size 0.8) (drill 0.4) (layers F.Cu B.Cu) (net 1))
-  (via (at 51 31) (size 0.8) (drill 0.4) (layers F.Cu B.Cu) (net 1))
-  (via (at 53 31) (size 0.8) (drill 0.4) (layers F.Cu B.Cu) (net 1))
+  (via (at 49 31.5) (size 0.8) (drill 0.4) (layers F.Cu B.Cu) (net 1))
   (via (at 55 31) (size 0.8) (drill 0.4) (layers F.Cu B.Cu) (net 1))
-  (via (at 57 31) (size 0.8) (drill 0.4) (layers F.Cu B.Cu) (net 1))
   (via (at 50 32.5) (size 0.8) (drill 0.4) (layers F.Cu B.Cu) (net 1))
   (via (at 52 32.5) (size 0.8) (drill 0.4) (layers F.Cu B.Cu) (net 1))
   (via (at 54 32.5) (size 0.8) (drill 0.4) (layers F.Cu B.Cu) (net 1))
-  (via (at 57 28) (size 0.8) (drill 0.4) (layers F.Cu B.Cu) (net 1))
+  (via (at 57 27.8) (size 0.8) (drill 0.4) (layers F.Cu B.Cu) (net 1))
   (via (at 58 27) (size 0.8) (drill 0.4) (layers F.Cu B.Cu) (net 1))
-  (via (at 60 31) (size 0.8) (drill 0.4) (layers F.Cu B.Cu) (net 1))
+  (via (at 60.7 31) (size 0.8) (drill 0.4) (layers F.Cu B.Cu) (net 1))
   (via (at 62 31) (size 0.8) (drill 0.4) (layers F.Cu B.Cu) (net 1))
   (via (at 64 31) (size 0.8) (drill 0.4) (layers F.Cu B.Cu) (net 1))
@@
   (via (at 40.8 30.2) (size 0.5) (drill 0.3) (layers F.Cu B.Cu) (net 1))
   (via (at 41.4 30.2) (size 0.5) (drill 0.3) (layers F.Cu B.Cu) (net 1))
+  (via (at 29.6 30.7) (size 0.8) (drill 0.4) (layers F.Cu B.Cu) (net 1))
+  (via (at 28.2 30.7) (size 0.8) (drill 0.4) (layers F.Cu B.Cu) (net 1))
+  (via (at 25.6 33.4) (size 0.8) (drill 0.4) (layers F.Cu B.Cu) (net 1))
+  (via (at 25.6 35) (size 0.8) (drill 0.4) (layers F.Cu B.Cu) (net 1))
+  (via (at 28.2 37.3) (size 0.8) (drill 0.4) (layers F.Cu B.Cu) (net 1))
+  (via (at 29.6 37.3) (size 0.8) (drill 0.4) (layers F.Cu B.Cu) (net 1))
+  (via (at 59.5 22.7) (size 0.8) (drill 0.4) (layers F.Cu B.Cu) (net 1))
+  (via (at 57.2 22.7) (size 0.8) (drill 0.4) (layers F.Cu B.Cu) (net 1))
+  (via (at 54.1 23) (size 0.8) (drill 0.4) (layers F.Cu B.Cu) (net 1))
+  (via (at 53.1 25) (size 0.8) (drill 0.4) (layers F.Cu B.Cu) (net 1))
+  (via (at 43 30) (size 0.8) (drill 0.4) (layers F.Cu B.Cu) (net 1))
+  (via (at 44.5 30) (size 0.8) (drill 0.4) (layers F.Cu B.Cu) (net 1))
+  (via (at 46 30) (size 0.8) (drill 0.4) (layers F.Cu B.Cu) (net 1))
+  (via (at 47.5 30) (size 0.8) (drill 0.4) (layers F.Cu B.Cu) (net 1))
+  (via (at 49 30) (size 0.8) (drill 0.4) (layers F.Cu B.Cu) (net 1))
+  (via (at 50.5 30) (size 0.8) (drill 0.4) (layers F.Cu B.Cu) (net 1))
   (segment (start 61.4625 24.9625) (end 61 24.5) (width 0.7) (layer F.Cu) (net 2))
   (segment (start 61.4625 27.5) (end 61.4625 24.9625) (width 0.7) (layer F.Cu) (net 2))
@@
     (polygon
       (pts
-        (xy 42.1 34.35) (xy 41.1 35.3) (xy 37.7 35.3) (xy 37.5 34.9) (xy 37.7 34.5)
-        (xy 40.8 34.5) (xy 41.9 33.275) (xy 41.9 31.1) (xy 40.5 31.1) (xy 40.5 32.85)
-        (xy 40.225 33.45) (xy 30.775 33.45) (xy 30 32.55) (xy 38.3 32.55) (xy 38.29375 33.05)
-        (xy 38.425 33.25) (xy 39.2 33.25) (xy 39.5 32.6) (xy 39.5 32.3) (xy 39.5 29.9)
-        (xy 42.1 29.9)
+        (xy 42.1 31) (xy 41.9 30.99375) (xy 41.9 30.5) (xy 40.5 30.5) (xy 40.5 32.85)
+        (xy 40.225 33.45) (xy 30.775 33.45) (xy 30 32.6) (xy 38.101563 32.625) (xy 38.1 33)
+        (xy 38.4125 33.3) (xy 39.5 33.3) (xy 39.5 29.9) (xy 42.1 29.9)
       )
     )
@@
     (polygon
       (pts
-        (xy 36.1 34.9) (xy 35.9 35.3) (xy 35.5 35.3) (xy 35.3 34.9) (xy 35.5 34.5)
-        (xy 35.9 34.5)
+        (xy 42.1 34.4) (xy 41.1 35.3) (xy 37.7 35.3) (xy 37.5 34.9) (xy 37.7 34.5)
+        (xy 40.8 34.5) (xy 42.1 33.2)
       )
     )
