File: PCB/Ampli/Ampli_IMS.sch (KiCad schematic (older format))
At the start: 15 parts, among them J1 5227161-3, J2 5227161-3, J3 Conn_01x03_Male, P1 300K, U1 LMC6082

Commit message: Update
Parts:
- C2, C5: LCSC (none) -> C360619
- C3, C4: LCSC (none) -> C139817
- D1, D2: LCSC (none) -> MSCD104H
- J1, J3, U1: LCSC (none) -> MOUSER
Changed lines of the file:
@@
 F 2 "Capacitor_Tantalum_SMD:CP_EIA-3216-18_Kemet-A_Pad1.58x1.35mm_HandSolder" H 4600 5800 50  0001 C CNN
 F 3 "~" H 4600 5800 50  0001 C CNN
+F 4 "C139817" H 4600 5800 50  0001 C CNN "LCSC"
 	1    4600 5800
 	1    0    0    -1
@@
 F 2 "Capacitor_Tantalum_SMD:CP_EIA-3216-18_Kemet-A_Pad1.58x1.35mm_HandSolder" H 4600 5400 50  0001 C CNN
 F 3 "~" H 4600 5400 50  0001 C CNN
+F 4 "C139817" H 4600 5400 50  0001 C CNN "LCSC"
 	1    4600 5400
 	1    0    0    -1
@@
 F 2 "Connector_Coaxial:SMA_Amphenol_132203-12_Horizontal" H 3250 3600 50  0001 C CNN
 F 3 "~" H 3250 3600 50  0001 C CNN
+F 4 "MOUSER" H 3250 3650 50  0001 C CNN "LCSC"
 	1    3250 3650
 	0    1    1    0
@@
 F 2 "Diode_SMD:D_0805_2012Metric_Castellated" H 4150 5250 50  0001 C CNN
 F 3 "~" H 4150 5250 50  0001 C CNN
+F 4 "MSCD104H" H 4150 5250 50  0001 C CNN "LCSC"
 	1    4150 5250
 	-1   0    0    1
@@
 F 2 "Diode_SMD:D_0805_2012Metric_Castellated" H 4150 5950 50  0001 C CNN
 F 3 "~" H 4150 5950 50  0001 C CNN
+F 4 "MSCD104H" H 4150 5950 50  0001 C CNN "LCSC"
 	1    4150 5950
 	1    0    0    -1
@@
 F 2 "Connector_JST:JST_EH_B3B-EH-A_1x03_P2.50mm_Vertical" H 3100 5600 50  0001 C CNN
 F 3 "~" H 3100 5600 50  0001 C CNN
+F 4 "MOUSER" H 3100 5600 50  0001 C CNN "LCSC"
 	1    3100 5600
 	1    0    0    -1
@@
 F 2 "Capacitor_SMD:C_0805_2012Metric" H 5850 6000 50  0001 C CNN
 F 3 "~" H 5850 6000 50  0001 C CNN
+F 4 "C360619" H 5850 6000 50  0001 C CNN "LCSC"
 	1    5850 6000
 	1    0    0    -1
@@
 F 2 "Package_SO:SO-8_3.9x4.9mm_P1.27mm" H 4200 3750 50  0001 C CNN
 F 3 "http://www.ti.com/lit/ds/symlink/lmc6082.pdf" H 4200 3750 50  0001 C CNN
+F 4 "MOUSER" H 4200 3750 50  0001 C CNN "LCSC"
 	1    4200 3750
 	1    0    0    1
@@
 F 2 "Package_SO:SO-8_3.9x4.9mm_P1.27mm" H 6350 3650 50  0001 C CNN
 F 3 "http://www.ti.com/lit/ds/symlink/lmc6082.pdf" H 6350 3650 50  0001 C CNN
+F 4 "MOUSER" H 6350 3650 50  0001 C CNN "LCSC"
 	2    6350 3650
 	1    0    0    1
@@
 F 2 "Package_SO:SO-8_3.9x4.9mm_P1.27mm" H 7350 5550 50  0001 C CNN
 F 3 "http://www.ti.com/lit/ds/symlink/lmc6082.pdf" H 7350 5550 50  0001 C CNN
+F 4 "MOUSER" H 7350 5550 50  0001 C CNN "LCSC"
 	3    7350 5550
 	1    0    0    -1
@@
 F 2 "Capacitor_SMD:C_0805_2012Metric" H 5850 5150 50  0001 C CNN
 F 3 "~" H 5850 5150 50  0001 C CNN
+F 4 "C360619" H 5850 5150 50  0001 C CNN "LCSC"
 	1    5850 5150
 	1    0    0    -1
