File: PCB/Electrodes/Electrodes/Electrodes.kicad_pcb (KiCad board)
At the start: 2 copper layers, 41 x 49 mm, 3 parts

Commit message: Update
Parts:
- removed REF**: Electrode_hole, Connector:Electrode_hole
- removed REF** (x2): Electrode_Pad, Connector:Electrode_Pad
- added J1: Conn_01x01_Female, Connector:Electrode_hole, F.Cu at (80.5, 105.5)
Routing:
- net GND: track 0.00 -> 98.1 mm
- net (no net): track 71.4 -> 0.00 mm
- added copper zone on B.Cu, net GND
- added copper zone on F.Cu, net GND
Other:
- board size 41 x 49 mm -> 41 x 48.5 mm
- board text added: "Electrode"
